File: Hardware/RevA/KiCad/MagniCube-RevA-LEDs.sch (KiCad schematic (older format))
At the start: 4 parts

Commit message: schematic in progress
Parts:
- added D_L0C0, D_L0C1, D_L0C10, D_L0C12, D_L0C13, D_L0C14, D_L0C15, D_L0C2, D_L0C3, D_L0C4, D_L0C5, D_L0C6, D_L0C7, D_L0C8, D_L0C9, D_L1C0, D_L1C1, D_L1C10, D_L1C11, D_L1C12, D_L1C13, D_L1C14, D_L1C15, D_L1C2, D_L1C3, D_L1C4, D_L1C5, D_L1C6, D_L1C7, D_L1C8, D_L1C9, D_L2C0, D_L2C1, D_L2C10, D_L2C11, D_L2C12, D_L2C13, D_L2C14, D_L2C15, D_L2C2, D_L2C3, D_L2C4, D_L2C5, D_L2C6, D_L2C7, D_L2C8, D_L2C9, D_L3C0, D_L3C1, D_L3C10, D_L3C11, D_L3C12, D_L3C13, D_L3C14, D_L3C15, D_L3C2, D_L3C3, D_L3C4, D_L3C5, D_L3C6, D_L3C7, D_L3C8, D_L3C9, D_l0C11: CUBE_LED, ~, symbol CUBE_LED
- added J_C0, J_C1, J_C10, J_C11, J_C12, J_C13, J_C14, J_C15, J_C2, J_C3, J_C4, J_C5, J_C6, J_C7, J_C8, J_C9: Column 0, ~, symbol HEADER_1
- added J_L0: Level 0, ~, symbol HEADER_1
- added J_L1: Level 1, ~, symbol HEADER_1
- added J_L2: Level 2, ~, symbol HEADER_1
- added J_L3: Level 3, ~, symbol HEADER_1
- renumbered R4 to R6, R5 to R7, R6 to R8, R7 to R9
Connections:
- wire segments 0 -> 24
Other:
- moved on the sheet: R6, R7, R8, R9

Commit message: PCB in progress
Parts:
- J_C1: value Column 0 -> Column 1
- J_C10: value Column 0 -> Column 10
- J_C11: value Column 0 -> Column 11
- J_C12: value Column 0 -> Column 12
- J_C13: value Column 0 -> Column 13
- J_C14: value Column 0 -> Column 14
- J_C15: value Column 0 -> Column 15
- J_C2: value Column 0 -> Column 2
- J_C3: value Column 0 -> Column 3
- J_C4: value Column 0 -> Column 4
- J_C5: value Column 0 -> Column 5
- J_C6: value Column 0 -> Column 6
- J_C7: value Column 0 -> Column 7
- J_C8: value Column 0 -> Column 8
- J_C9: value Column 0 -> Column 9
Changed lines of the file:
@@
 Sheet 4 4
 Title ""
-Date "14 apr 2016"
+Date "18 apr 2016"
 Rev ""
 Comp ""
@@
 P 4000 4150
 F 0 "J_C1" H 4000 4300 60  0000 C TNN
-F 1 "Column 0" H 4000 4000 60  0001 C CNN
+F 1 "Column 1" H 4000 4000 60  0001 C CNN
 F 2 "~" H 4000 4150 60  0000 C CNN
 F 3 "~" H 4000 4150 60  0000 C CNN
@@
 P 4800 4150
 F 0 "J_C3" H 4800 4300 60  0000 C TNN
-F 1 "Column 0" H 4800 4000 60  0001 C CNN
+F 1 "Column 3" H 4800 4000 60  0001 C CNN
 F 2 "~" H 4800 4150 60  0000 C CNN
 F 3 "~" H 4800 4150 60  0000 C CNN
@@
 P 5200 4150
 F 0 "J_C4" H 5200 4300 60  0000 C TNN
-F 1 "Column 0" H 5200 4000 60  0001 C CNN
+F 1 "Column 4" H 5200 4000 60  0001 C CNN
 F 2 "~" H 5200 4150 60  0000 C CNN
 F 3 "~" H 5200 4150 60  0000 C CNN
@@
 P 5600 4150
 F 0 "J_C5" H 5600 4300 60  0000 C TNN
-F 1 "Column 0" H 5600 4000 60  0001 C CNN
+F 1 "Column 5" H 5600 4000 60  0001 C CNN
 F 2 "~" H 5600 4150 60  0000 C CNN
 F 3 "~" H 5600 4150 60  0000 C CNN
@@
 P 6000 4150
 F 0 "J_C6" H 6000 4300 60  0000 C TNN
-F 1 "Column 0" H 6000 4000 60  0001 C CNN
+F 1 "Column 6" H 6000 4000 60  0001 C CNN
 F 2 "~" H 6000 4150 60  0000 C CNN
 F 3 "~" H 6000 4150 60  0000 C CNN
@@
 P 6400 4150
 F 0 "J_C7" H 6400 4300 60  0000 C TNN
-F 1 "Column 0" H 6400 4000 60  0001 C CNN
+F 1 "Column 7" H 6400 4000 60  0001 C CNN
 F 2 "~" H 6400 4150 60  0000 C CNN
 F 3 "~" H 6400 4150 60  0000 C CNN
@@
 P 6800 4150
 F 0 "J_C8" H 6800 4300 60  0000 C TNN
-F 1 "Column 0" H 6800 4000 60  0001 C CNN
+F 1 "Column 8" H 6800 4000 60  0001 C CNN
 F 2 "~" H 6800 4150 60  0000 C CNN
 F 3 "~" H 6800 4150 60  0000 C CNN
@@
 P 7200 4150
 F 0 "J_C9" H 7200 4300 60  0000 C TNN
-F 1 "Column 0" H 7200 4000 60  0001 C CNN
+F 1 "Column 9" H 7200 4000 60  0001 C CNN
 F 2 "~" H 7200 4150 60  0000 C CNN
 F 3 "~" H 7200 4150 60  0000 C CNN
@@
 P 7600 4150
 F 0 "J_C10" H 7600 4300 60  0000 C TNN
-F 1 "Column 0" H 7600 4000 60  0001 C CNN
+F 1 "Column 10" H 7600 4000 60  0001 C CNN
 F 2 "~" H 7600 4150 60  0000 C CNN
 F 3 "~" H 7600 4150 60  0000 C CNN
@@
 P 8000 4150
 F 0 "J_C11" H 8000 4300 60  0000 C TNN
-F 1 "Column 0" H 8000 4000 60  0001 C CNN
+F 1 "Column 11" H 8000 4000 60  0001 C CNN
 F 2 "~" H 8000 4150 60  0000 C CNN
 F 3 "~" H 8000 4150 60  0000 C CNN
@@
 P 8400 4150
 F 0 "J_C12" H 8400 4300 60  0000 C TNN
-F 1 "Column 0" H 8400 4000 60  0001 C CNN
+F 1 "Column 12" H 8400 4000 60  0001 C CNN
 F 2 "~" H 8400 4150 60  0000 C CNN
 F 3 "~" H 8400 4150 60  0000 C CNN
@@
 P 8800 4150
 F 0 "J_C13" H 8800 4300 60  0000 C TNN
-F 1 "Column 0" H 8800 4000 60  0001 C CNN
+F 1 "Column 13" H 8800 4000 60  0001 C CNN
 F 2 "~" H 8800 4150 60  0000 C CNN
 F 3 "~" H 8800 4150 60  0000 C CNN
@@
 P 9200 4150
 F 0 "J_C14" H 9200 4300 60  0000 C TNN
-F 1 "Column 0" H 9200 4000 60  0001 C CNN
+F 1 "Column 14" H 9200 4000 60  0001 C CNN
 F 2 "~" H 9200 4150 60  0000 C CNN
 F 3 "~" H 9200 4150 60  0000 C CNN
@@
 P 9600 4150
 F 0 "J_C15" H 9600 4300 60  0000 C TNN
-F 1 "Column 0" H 9600 4000 60  0001 C CNN
+F 1 "Column 15" H 9600 4000 60  0001 C CNN
 F 2 "~" H 9600 4150 60  0000 C CNN
 F 3 "~" H 9600 4150 60  0000 C CNN
@@
 P 4400 4150
 F 0 "J_C2" H 4400 4300 60  0000 C TNN
-F 1 "Column 0" H 4400 4000 60  0001 C CNN
+F 1 "Column 2" H 4400 4000 60  0001 C CNN
 F 2 "~" H 4400 4150 60  0000 C CNN
 F 3 "~" H 4400 4150 60  0000 C CNN

Commit message: work in progress
Parts:
- renumbered R6 to R4, R7 to R5, R8 to R6, R9 to R7
Changed lines of the file:
@@
 Sheet 4 4
 Title ""
-Date "18 apr 2016"
+Date "19 apr 2016"
 Rev ""
 Comp ""
@@
 LED_C15
 $Comp
-L R R6
+L R R4
 U 1 1 570451BA
 P 2700 2300
-F 0 "R6" V 2780 2300 40  0000 C CNN
+F 0 "R4" V 2780 2300 40  0000 C CNN
 F 1 "270" V 2707 2301 40  0000 C CNN
 F 2 "~" V 2630 2300 30  0000 C CNN
@@
 $EndComp
 $Comp
-L R R7
+L R R5
 U 1 1 570451D8
 P 2700 2700
-F 0 "R7" V 2780 2700 40  0000 C CNN
+F 0 "R5" V 2780 2700 40  0000 C CNN
 F 1 "270" V 2707 2701 40  0000 C CNN
 F 2 "~" V 2630 2700 30  0000 C CNN
@@
 $EndComp
 $Comp
-L R R8
+L R R6
 U 1 1 570451DE
 P 2700 3100
-F 0 "R8" V 2780 3100 40  0000 C CNN
+F 0 "R6" V 2780 3100 40  0000 C CNN
 F 1 "270" V 2707 3101 40  0000 C CNN
 F 2 "~" V 2630 3100 30  0000 C CNN
@@
 $EndComp
 $Comp
-L R R9
+L R R7
 U 1 1 570451E4
 P 2700 3500
-F 0 "R9" V 2780 3500 40  0000 C CNN
+F 0 "R7" V 2780 3500 40  0000 C CNN
 F 1 "270" V 2707 3501 40  0000 C CNN
 F 2 "~" V 2630 3500 30  0000 C CNN
