File: Hardware/RevA/KiCad/MagniCube-RevA.kicad_pcb (KiCad board)
At the start: 2 copper layers, 50 x 50 mm, 61 parts, among them CON1 USB-MINI-B, CON2 DC_JACK, CON3 BDM, IC1 FT232RL, IC2 MC9S12VR64, IC3 MC9S12VRP64

Commit message: work in progress
Parts:
- added SG: 0.6, spark_gap_pad_0.6, F.Cu at (128.3, 113.7)
- added SG: 0.6, spark_gap_pad_0.6, F.Cu at (127.7, 113.7)
- added SG: 0.6, spark_gap_pad_0.6, F.Cu at (122.7, 124.3)
- added SG: 0.6, spark_gap_pad_0.6, F.Cu at (122.1, 124.3)
- added SG: 0.6, spark_gap_pad_0.6, F.Cu at (122.1, 110.3)
- added SG: 0.6, spark_gap_pad_0.6, F.Cu at (122.7, 110.3)
- added SG: 0.6, spark_gap_pad_0.6, F.Cu at (122.1, 99.7)
- added SG: 0.6, spark_gap_pad_0.6, F.Cu at (122.7, 99.7)
- added SG: 0.6, spark_gap_pad_0.6, F.Cu at (122.1, 85.7)
- added SG: 0.6, spark_gap_pad_0.6, F.Cu at (122.7, 85.7)
- added SG: 0.6, spark_gap_pad_0.6, F.Cu at (161.7, 113.7)
- added SG: 0.6, spark_gap_pad_0.6, F.Cu at (148.7, 113.7)
- added SG: 0.6, spark_gap_pad_0.6, F.Cu at (162.3, 113.7)
- added SG: 0.6, spark_gap_pad_0.6, F.Cu at (148.1, 113.7)
- added SG: 0.6, spark_gap_pad_0.6, F.Cu at (141.3, 113.7)
- added SG: 0.6, spark_gap_pad_0.6, F.Cu at (141.9, 113.7)
- C10: value 4.7uF -> 100nf
- IC2: moved to B.Cu
- R2: value 100 -> 10k
- R3: value 100 -> 4k7
- R4: value 10k -> 270; moved to F.Cu
- R5: value 4k7 -> 270
- R6, R7: moved to F.Cu
- moved C7 47.4 mm to (138.0, 103.8), turned to 90 degrees
- moved FB1 40.0 mm to (104.0, 144.0)
- moved R5 37.8 mm to (139.7, 112.7), turned to 90 degrees
- moved R7 30.9 mm to (160.1, 112.7), turned to 90 degrees
- moved IC2 29.7 mm to (130.9, 103.8), turned to 135 degrees
- moved R6 29.5 mm to (150.3, 112.7), turned to 90 degrees
- moved SG 29.2 mm to (115.1, 104.7)
- moved SG 29.2 mm to (115.7, 104.7)
- moved SG 29.2 mm to (116.2, 104.7)
- moved PIN_STRIP_3x2-90 23.8 mm to (108.0, 99.0)
- moved C5 22.1 mm to (113.0, 118.0)
- moved R4 20.4 mm to (129.9, 112.7)
- moved J_L0 14.0 mm to (124.0, 112.0)
- moved J_L1 14.0 mm to (138.0, 112.0)
- moved J_L2 14.0 mm to (153.0, 112.0)
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Connections:
- C1 pad 1: 5V -> N-0000098
- C1 pad 2: GND -> N-0000087
- C10 pad 1: 5V -> N-0000036
- C10 pad 2: GND -> N-0000035
- C11 pad 1: 5V -> N-0000036
- C11 pad 2: GND -> N-0000035
- C2 pad 1: 5V -> N-0000098
- C2 pad 2: GND -> N-0000087
- C3 pad 1: 5V -> N-0000098
- C3 pad 2: GND -> N-0000087
- C4 pad 2: GND -> (no net)
- C5 pad 1: GND -> (no net)
- C6 pad 1: 5V -> N-0000036
- C6 pad 2: GND -> N-0000035
- C7 pad 1: 5V -> N-0000036
- C7 pad 2: GND -> N-0000035
- C8 pad 1: 5V -> N-0000036
- C8 pad 2: GND -> N-0000035
- CON1 pad 5: GND -> (no net)
- CON2 pad 1: GND -> N-0000032
- CON2 pad 2: GND -> N-0000032
- CON2 pad 3: 12V -> (no net)
- CON3 pad 2: GND -> (no net)
- CON3 pad 6: 5V -> (no net)
- D_RXTX1 pad 1: 5V -> (no net)
- D_VUSB1 pad 1: N-0000069 (its old number) -> N-0000094
- D_VUSB1 pad 2: 12V -> (no net)
- FB1 pad 2: N-0000069 (its old number) -> N-0000094
- IC1 pad 1: N-0000074 -> UART_RXD
- IC1 pad 18: GND -> N-00000105
- IC1 pad 19: N-0000081 -> N-00000107
- IC1 pad 20: 5V -> N-00000100
- IC1 pad 21: GND -> N-00000105
- IC1 pad 25: GND -> N-00000105
- IC1 pad 26: GND -> N-00000105
- IC1 pad 4: 5V -> N-00000100
- IC1 pad 5: N-0000072 -> UART_TXD
- IC1 pad 7: GND -> N-00000105
- IC2 pad 13: GND -> (no net)
- IC2 pad 18: GND -> (no net)
- IC2 pad 21: 5V -> (no net)
- IC2 pad 25: 12V -> N-0000073
- IC2 pad 26: 12V -> N-0000073
- IC2 pad 28: GND -> (no net)
- IC2 pad 37: 5V -> (no net)
- IC2 pad 38: GND -> (no net)
- IC2 pad 7: 5V -> (no net)
- IC3 pad 13: GND -> (no net)
- IC3 pad 18: GND -> (no net)
- IC3 pad 21: 5V -> (no net)
- IC3 pad 25: 12V -> (no net)
- IC3 pad 27: GND -> (no net)
- IC3 pad 37: 5V -> (no net)
- IC3 pad 38: GND -> (no net)
- IC3 pad 8: 5V -> (no net)
- J_L0 pad 1: N-0000085 -> N-00000112
- J_L1 pad 1: N-0000086 -> N-00000113
- J_L2 pad 1: N-0000088 -> N-00000115
- J_L3 pad 1: N-0000087 -> N-00000114
- R2 pad 1: UART_RXD -> N-00000107
- R2 pad 2: N-0000074 -> (no net)
- R3 pad 1: UART_TXD -> N-0000094
- R3 pad 2: N-0000072 -> N-00000107
- R4 pad 1: N-0000081 -> LED_L0
- R4 pad 2: GND -> N-00000112
- R5 pad 1: N-0000069 (its old number) -> LED_L1
- R5 pad 2: N-0000081 -> N-00000113
- R6 pad 1: LED_L0 -> LED_L2
- R6 pad 2: N-0000085 -> N-00000115
- R7 pad 1: LED_L1 -> LED_L3
- R7 pad 2: N-0000086 -> N-00000114
Routing:
- net LED_C0: track 0.00 -> 42.5 mm, vias 0 -> 1
- net LED_C3: track 0.00 -> 40.1 mm, vias 0 -> 1
- net LED_L3: track 0.00 -> 32.0 mm, vias 0 -> 1
- net LED_C1: track 0.00 -> 29.0 mm, vias 0 -> 1
- net LED_C2: track 0.00 -> 28.8 mm, vias 0 -> 1
- net LED_L0: track 0.00 -> 23.4 mm, vias 0 -> 1
- net LED_L2: track 0.00 -> 22.3 mm, vias 0 -> 1
- net LED_L1: track 0.00 -> 15.1 mm, vias 0 -> 1
- net LED_C4: track 0.00 -> 4.55 mm
- net N-00000115: track 0.00 -> 3.53 mm
- net N-00000113: track 0.00 -> 3.53 mm
- net N-00000114: track 0.00 -> 3.52 mm
- net N-00000112: track 0.00 -> 3.52 mm
Other:
- net class Default: clearance 0.25 -> 0.2
- net class Power added: clearance 0.2, trace_width 0.4, via_dia 0.8, via_drill 0.3
- rule trace_clearance: 0.25 -> 0.2

Commit message: work in progress
Parts:
- added SG: 0.6, spark_gap_pad_0.6, B.Cu at (138.1, 113.7)
- added SG: 0.6, spark_gap_pad_0.6, B.Cu at (137.5, 113.7)
- C6, R5, SG (x2): moved to B.Cu
- moved C6 51.3 mm to (138.0, 104.5), turned to 90 degrees
- moved C7 0.70 mm to (138.0, 104.5)
Connections:
- C1 pad 1: N-0000098 -> /UART/5V
- C1 pad 2: N-0000087 -> /UART/GND
- C10 pad 1: N-0000036 -> /MCU/5V
- C10 pad 2: N-0000035 -> /MCU/GND
- C11 pad 1: N-0000036 -> /MCU/5V
- C11 pad 2: N-0000035 -> /MCU/GND
- C2 pad 1: N-0000098 -> /UART/5V
- C2 pad 2: N-0000087 -> /UART/GND
- C3 pad 1: N-0000098 -> /UART/5V
- C3 pad 2: N-0000087 -> /UART/GND
- C4 pad 2: (no net) -> /UART/GND
- C5 pad 1: (no net) -> /UART/GND
- C6 pad 1: N-0000036 -> /MCU/5V
- C6 pad 2: N-0000035 -> /MCU/GND
- C7 pad 1: N-0000036 -> /MCU/5V
- C7 pad 2: N-0000035 -> /MCU/GND
- C8 pad 1: N-0000036 -> /MCU/5V
- C8 pad 2: N-0000035 -> /MCU/GND
- CON1 pad 5: (no net) -> /UART/GND
- CON2 pad 1: N-0000032 -> /MCU/GND
- CON2 pad 2: N-0000032 -> /MCU/GND
- CON2 pad 3: (no net) -> /MCU/12V
- CON3 pad 2: (no net) -> /MCU/GND
- D_RXTX1 pad 1: (no net) -> /UART/5V
- IC1 pad 18: N-00000105 -> /UART/GND
- IC1 pad 20: N-00000100 -> /UART/5V
- IC1 pad 21: N-00000105 -> /UART/GND
- IC1 pad 25: N-00000105 -> /UART/GND
- IC1 pad 26: N-00000105 -> /UART/GND
- IC1 pad 4: N-00000100 -> /UART/5V
- IC1 pad 7: N-00000105 -> /UART/GND
- IC2 pad 1: N-0000069 -> /MCU/GND
- IC2 pad 13: (no net) -> /MCU/GND
- IC2 pad 18: (no net) -> /MCU/GND
- IC2 pad 21: (no net) -> /MCU/5V
- IC2 pad 25: N-0000073 -> /MCU/12V
- IC2 pad 26: N-0000073 -> /MCU/12V
- IC2 pad 28: (no net) -> /MCU/GND
- IC2 pad 37: (no net) -> /MCU/5V
- IC2 pad 38: (no net) -> /MCU/GND
- IC2 pad 4: N-0000069 -> /MCU/GND
- IC2 pad 6: N-0000069 -> /MCU/GND
- IC2 pad 7: (no net) -> /MCU/5V
- IC3 pad 1: N-0000070 -> /MCU/GND
- IC3 pad 13: (no net) -> /MCU/GND
- IC3 pad 18: (no net) -> /MCU/GND
- IC3 pad 21: (no net) -> /MCU/5V
- IC3 pad 25: (no net) -> /MCU/12V
- IC3 pad 27: (no net) -> /MCU/GND
- IC3 pad 37: (no net) -> /MCU/5V
- IC3 pad 38: (no net) -> /MCU/GND
- IC3 pad 4: N-0000070 -> /MCU/GND
- IC3 pad 7: N-0000070 -> /MCU/GND
- IC3 pad 8: (no net) -> /MCU/5V
- J_L0 pad 1: N-00000112 -> N-0000085
- J_L2 pad 1: N-00000115 -> N-0000088
- J_L3 pad 1: N-00000114 -> N-0000087
- R2 pad 2: (no net) -> /UART/GND
- R4 pad 2: N-00000112 -> N-0000085
- R6 pad 2: N-00000115 -> N-0000088
- R7 pad 2: N-00000114 -> N-0000087
Routing:
- net LED_C4: track 4.55 -> 32.3 mm, vias 0 -> 2
- net LED_C5: track 0.00 -> 26.2 mm, vias 0 -> 1
- net /MCU/5V: track 0.00 -> 5.48 mm, vias 0 -> 1
- net N-0000087: track 0.00 -> 2.31 mm
- net N-00000114: track 3.52 -> 1.21 mm
- net N-0000088: track 0.00 -> 1.98 mm
- net N-00000115: track 3.53 -> 1.55 mm
- net N-0000085: track 0.00 -> 1.97 mm
- net N-00000112: track 3.52 -> 1.55 mm
- net LED_L1: vias 1 -> 2
- net /MCU/GND: vias 0 -> 1

Commit message: work in progress
Parts:
- removed the SG at (115.1, 104.7)
- removed the SG at (128.3, 113.7)
- removed the SG at (127.7, 113.7)
- removed the SG at (122.7, 124.3)
- removed the SG at (122.1, 124.3)
- removed the SG at (122.1, 110.3)
- removed the SG at (122.7, 110.3)
- removed the SG at (122.1, 99.7)
- removed the SG at (122.7, 99.7)
- removed the SG at (122.1, 85.7)
- removed the SG at (122.7, 85.7)
- removed the SG at (115.7, 104.7)
- removed the SG at (138.1, 113.7)
- removed the SG at (137.5, 113.7)
- removed the SG at (116.2, 104.7)
- removed the SG at (161.7, 113.7)
- removed the SG at (148.7, 113.7)
- removed the SG at (162.3, 113.7)
- removed the SG at (148.1, 113.7)
- removed the SG at (141.3, 113.7)
- removed the SG at (141.9, 113.7)
- added SG: 1.0, spark_gap_pad_1.0, B.Cu at (141.8, 114.7)
- added SG: 1.0, spark_gap_pad_1.0, B.Cu at (121.8, 110.3)
- added SG: 1.0, spark_gap_pad_1.0, B.Cu at (122.8, 109.3)
- added SG: 1.0, spark_gap_pad_1.0, B.Cu at (122.8, 110.3)
- added SG: 1.0, spark_gap_pad_1.0, B.Cu at (122.8, 99.7)
- added SG: 1.0, spark_gap_pad_1.0, B.Cu at (121.8, 99.7)
- added SG: 1.0, spark_gap_pad_1.0, B.Cu at (122.8, 100.7)
- added SG: 1.0, spark_gap_pad_1.0, B.Cu at (122.8, 85.7)
- added SG: 1.0, spark_gap_pad_1.0, B.Cu at (122.8, 86.7)
- added SG: 1.0, spark_gap_pad_1.0, B.Cu at (121.8, 85.7)
- added SG: 1.0, spark_gap_pad_1.0, B.Cu at (122.8, 123.3)
- added SG: 1.0, spark_gap_pad_1.0, B.Cu at (141.8, 113.7)
- added SG: 1.0, spark_gap_pad_1.0, B.Cu at (122.8, 124.3)
- added SG: 1.0, spark_gap_pad_1.0, B.Cu at (121.8, 124.3)
- added SG: 1.0, spark_gap_pad_1.0, B.Cu at (135.0, 126.0)
- added SG: 1.0, spark_gap_pad_1.0, B.Cu at (135.0, 127.0)
- added SG: 1.0, spark_gap_pad_1.0, B.Cu at (134.0, 126.0)
- added SG: 1.0, spark_gap_pad_1.0, B.Cu at (148.2, 114.7)
- added SG: 1.0, spark_gap_pad_1.0, B.Cu at (148.2, 113.7)
- added SG: 1.0, spark_gap_pad_1.0, B.Cu at (147.2, 113.7)
- added SG: 1.0, spark_gap_pad_1.0, B.Cu at (162.2, 113.7)
- added SG: 1.0, spark_gap_pad_1.0, B.Cu at (163.2, 113.7)
- added SG: 1.0, spark_gap_pad_1.0, B.Cu at (136.7, 114.7)
- added SG: 1.0, spark_gap_pad_1.0, B.Cu at (162.2, 114.7)
- added SG: 1.0, spark_gap_pad_1.0, B.Cu at (136.8, 100.7)
- added SG: 1.0, spark_gap_pad_1.0, B.Cu at (137.8, 99.7)
- added SG: 1.0, spark_gap_pad_1.0, B.Cu at (136.8, 99.7)
- added SG: 1.0, spark_gap_pad_1.0, B.Cu at (136.8, 85.7)
- added SG: 1.0, spark_gap_pad_1.0, B.Cu at (135.8, 85.7)
- added SG: 1.0, spark_gap_pad_1.0, B.Cu at (136.8, 86.7)
- added SG: 1.0, spark_gap_pad_1.0, B.Cu at (153.2, 85.7)
- added SG: 1.0, spark_gap_pad_1.0, B.Cu at (153.2, 86.7)
- added SG: 1.0, spark_gap_pad_1.0, B.Cu at (154.2, 85.7)
- added SG: 1.0, spark_gap_pad_1.0, B.Cu at (142.8, 113.7)
- added SG: 1.0, spark_gap_pad_1.0, B.Cu at (167.2, 85.7)
- added SG: 1.0, spark_gap_pad_1.0, B.Cu at (167.2, 86.7)
- added SG: 1.0, spark_gap_pad_1.0, B.Cu at (168.2, 85.7)
- added SG: 1.0, spark_gap_pad_1.0, B.Cu at (167.2, 99.7)
- added SG: 1.0, spark_gap_pad_1.0, B.Cu at (168.2, 99.7)
- added SG: 1.0, spark_gap_pad_1.0, B.Cu at (167.2, 100.7)
- added SG: 1.0, spark_gap_pad_1.0, B.Cu at (168.2, 113.7)
- added SG: 1.0, spark_gap_pad_1.0, B.Cu at (167.2, 114.7)
- added SG: 1.0, spark_gap_pad_1.0, B.Cu at (167.2, 113.7)
- added SG: 1.0, spark_gap_pad_1.0, B.Cu at (167.2, 124.3)
- added SG: 1.0, spark_gap_pad_1.0, B.Cu at (137.7, 113.7)
- added SG: 1.0, spark_gap_pad_1.0, B.Cu at (168.2, 124.3)
- added SG: 1.0, spark_gap_pad_1.0, B.Cu at (167.2, 123.3)
- added SG: 1.0, spark_gap_pad_1.0, B.Cu at (154.2, 99.7)
- added SG: 1.0, spark_gap_pad_1.0, B.Cu at (153.2, 99.7)
- added SG: 1.0, spark_gap_pad_1.0, B.Cu at (153.2, 100.7)
- added SG: 1.0, spark_gap_pad_1.0, B.Cu at (153.2, 114.7)
- added SG: 1.0, spark_gap_pad_1.0, B.Cu at (154.2, 113.7)
- added SG: 1.0, spark_gap_pad_1.0, B.Cu at (153.2, 113.7)
- added SG: 1.0, spark_gap_pad_1.0, B.Cu at (155.0, 127.0)
- added SG: 1.0, spark_gap_pad_1.0, B.Cu at (155.0, 126.0)
- added SG: 1.0, spark_gap_pad_1.0, B.Cu at (136.7, 113.7)
- added SG: 1.0, spark_gap_pad_1.0, B.Cu at (156.0, 126.0)
- added SG: 1.0, spark_gap_pad_1.0, B.Cu at (145.5, 92.0)
- added SG: 1.0, spark_gap_pad_1.0, B.Cu at (149.3, 88.3)
- added SG: 1.0, spark_gap_pad_1.0, B.Cu at (146.5, 92.0)
- added SG: 1.0, spark_gap_pad_1.0, B.Cu at (149.3, 89.3)
- added SG: 1.0, spark_gap_pad_1.0, F.Cu at (140.0, 90.9)
- added SG: 1.0, spark_gap_pad_1.0, B.Cu at (149.3, 90.3)
- added SG: 1.0, spark_gap_pad_1.0, B.Cu at (126.8, 113.7)
- added SG: 1.0, spark_gap_pad_1.0, B.Cu at (127.8, 114.7)
- added SG: 1.0, spark_gap_pad_1.0, B.Cu at (127.8, 113.7)
- C8, R4, R6, R7: moved to B.Cu
- moved dc_socket_rh 90.2 mm to (183.3, 110.0), turned to 90 degrees
- moved C8 44.4 mm to (146.2, 101.8), turned to 90 degrees
- moved CON3 34.0 mm to (145.0, 89.3), turned to 180 degrees
- moved R8 29.1 mm to (179.5, 98.1)
- moved R3 27.6 mm to (183.6, 124.8)
- moved CON2 24.9 mm to (162.7, 105.0), turned to 90 degrees
- moved R2 20.8 mm to (178.6, 122.8)
- moved R9 19.3 mm to (181.3, 101.7)
- moved PIN_STRIP_3x2-90 8.46 mm to (110.1, 90.8), turned to 180 degrees
- moved J_L2 4.81 mm to (148.2, 112.0)
- moved J_L3 4.81 mm to (162.2, 112.0)
- moved J_L0 3.81 mm to (127.8, 112.0)
- moved J_L1 3.81 mm to (141.8, 112.0)
- moved J_C10 1.27 mm to (153.3, 98.0)
- moved J_C11 1.27 mm to (153.3, 84.0)
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Routing:
- net LED_C14: track 0.00 -> 41.3 mm, vias 0 -> 1
- net /MCU/BKGD: track 0.00 -> 37.0 mm, vias 0 -> 1
- net /MCU/RESET: track 0.00 -> 36.0 mm, vias 0 -> 1
- net LED_C11: track 0.00 -> 32.8 mm, vias 0 -> 1
- net LED_C15: track 0.00 -> 31.1 mm, vias 0 -> 1
- net LED_C7: track 0.00 -> 31.0 mm, vias 0 -> 1
- net LED_C12: track 0.00 -> 30.5 mm, vias 0 -> 1
- net /MCU/5V: track 5.48 -> 34.5 mm, vias 1 -> 3
- net LED_C13: track 0.00 -> 28.4 mm, vias 0 -> 1
- net LED_C6: track 0.00 -> 27.6 mm, vias 0 -> 1
- net UART_TXD: track 0.00 -> 27.5 mm, vias 0 -> 1
- net UART_RXD: track 0.00 -> 25.7 mm, vias 0 -> 1
- net LED_C8: track 0.00 -> 25.1 mm, vias 0 -> 1
- net LED_C9: track 0.00 -> 22.3 mm, vias 0 -> 1
- net LED_C10: track 0.00 -> 18.7 mm, vias 0 -> 1
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Other:
- outline, holes or cut-outs redrawn

Commit message: work in progress
Parts:
- removed C12: 100nf, c_0805
- removed C13: C, c_0805
- removed D_VUSB1: SCHOTTKY, diode_do35
- removed the SG at (136.8, 99.7)
- added D1: SCHOTTKY, sod80c, B.Cu at (153.7, 105.0)
- added D2: SCHOTTKY, sod80c, F.Cu at (170.1, 130.1)
- added SG: 1.0, spark_gap_pad_1.0, B.Cu at (135.0, 98.0)
- added SG: 1.0, spark_gap_pad_1.0, B.Cu at (140.4, 91.9)
- added SG: 1.0, spark_gap_pad_1.0, B.Cu at (140.4, 90.9)
- added SG: 1.0, spark_gap_pad_1.0, B.Cu at (139.4, 91.9)
- C9: value C -> 100nf; moved to B.Cu
- SG: moved to B.Cu
- moved C11 56.1 mm to (129.8, 105.4), turned to 180 degrees
- moved C10 43.6 mm to (130.0, 102.0), turned to 90 degrees
- moved C9 37.6 mm to (146.6, 105.2)
- moved C2 36.1 mm to (137.7, 142.0)
- moved C3 29.5 mm to (144.1, 142.1)
- moved SG 10.9 mm to (150.6, 88.5)
- moved SG 4.10 mm to (149.6, 91.9)
- moved SG 4.10 mm to (150.6, 91.9)
- moved SG 3.89 mm to (134.0, 98.0)
- moved SG 2.89 mm to (135.0, 99.0)
- moved SG 0.85 mm to (149.6, 87.5)
- moved SG 0.85 mm to (149.6, 88.5)
- moved SG 0.67 mm to (149.6, 90.9)
- moved C8 0.36 mm to (145.9, 102.0)
Connections:
- C9 pad 1: 12V -> /MCU/5V
- C9 pad 2: GND -> /MCU/GND
- CON2 pad 3: /MCU/12V -> N-000004
- CON3 pad 6: (no net) -> /MCU/5V
- SG pad : (no net) -> GND
Routing:
- net /MCU/BKGD: track 37.0 -> 58.2 mm
- net LED_C11: track 32.8 -> 53.5 mm
- net LED_C7: track 31.0 -> 51.3 mm, vias 1 -> 2
- net LED_C6: track 27.6 -> 46.3 mm
- net /MCU/5V: track 34.5 -> 52.5 mm, vias 3 -> 6
- net /MCU/12V: track 9.90 -> 26.4 mm, vias 0 -> 1
- net /MCU/RESET: track 36.0 -> 51.4 mm
- net LED_C10: track 18.7 -> 28.3 mm
- net LED_C12: track 30.5 -> 39.5 mm
- net LED_C13: track 28.4 -> 36.3 mm
- net LED_C3: track 38.6 -> 44.0 mm
- net N-000004: track 0.00 -> 4.62 mm
- net LED_C2: track 28.8 -> 32.6 mm

Commit message: work in progress
Parts:
- removed PIN_STRIP_3x2-90: Val**, pin_strip_3x2-90_with_dimensions
- removed R8, R9: 270, r_0805
- removed the SG at (167.2, 124.3)
- removed the SG at (168.2, 124.3)
- removed VIA: GND, via
- removed dc_socket_rh: VAL**, dc_socket_rh_with_dimensions
- added SG: 1.0, spark_gap_pad_1.0, B.Cu at (168.0, 124.3)
- added SG: 1.0, spark_gap_pad_1.0, B.Cu at (167.0, 124.3)
- moved C5 52.2 mm to (163.1, 133.0)
- moved FB1 43.6 mm to (146.5, 134.2)
- moved C1 5.42 mm to (151.2, 136.7)
- moved D2 4.71 mm to (171.4, 134.6)
- moved SG 2.00 mm to (166.2, 99.7)
- moved SG 1.90 mm to (166.3, 113.7)
- moved SG 1.90 mm to (152.3, 113.7)
- moved SG 0.80 mm to (168.0, 123.3)
- moved SG 0.10 mm to (167.3, 114.7)
- moved SG 0.10 mm to (167.3, 113.7)
- moved SG 0.10 mm to (153.3, 114.7)
- moved SG 0.10 mm to (153.3, 113.7)
Connections:
- C1 pad 1: /UART/5V -> 5V
- C1 pad 2: /UART/GND -> GND
- C10 pad 1: /MCU/5V -> 5V
- C10 pad 2: /MCU/GND -> GND
- C11 pad 1: /MCU/5V -> 5V
- C11 pad 2: /MCU/GND -> GND
- C2 pad 1: /UART/5V -> 5V
- C2 pad 2: /UART/GND -> GND
- C3 pad 1: /UART/5V -> 5V
- C3 pad 2: /UART/GND -> GND
- C4 pad 2: /UART/GND -> GND
- C5 pad 1: /UART/GND -> GND
- C6 pad 1: /MCU/5V -> 5V
- C6 pad 2: /MCU/GND -> GND
- C7 pad 1: /MCU/5V -> 5V
- C7 pad 2: /MCU/GND -> GND
- C8 pad 1: /MCU/5V -> 5V
- C8 pad 2: /MCU/GND -> GND
- C9 pad 1: /MCU/5V -> 5V
- C9 pad 2: /MCU/GND -> GND
- CON1 pad 5: /UART/GND -> GND
- CON2 pad 1: /MCU/GND -> GND
- CON2 pad 2: /MCU/GND -> GND
- CON3 pad 2: /MCU/GND -> GND
- CON3 pad 6: /MCU/5V -> 5V
- D1 pad 2: /MCU/12V -> 12V
- D2 pad 2: (no net) -> 12V
- D_RXTX1 pad 1: /UART/5V -> 5V
- IC1 pad 18: /UART/GND -> GND
- IC1 pad 20: /UART/5V -> 5V
- IC1 pad 21: /UART/GND -> GND
- IC1 pad 25: /UART/GND -> GND
- IC1 pad 26: /UART/GND -> GND
- IC1 pad 4: /UART/5V -> 5V
- IC1 pad 7: /UART/GND -> GND
- IC2 pad 1: /MCU/GND -> GND
- IC2 pad 13: /MCU/GND -> GND
- IC2 pad 18: /MCU/GND -> GND
- IC2 pad 21: /MCU/5V -> 5V
- IC2 pad 25: /MCU/12V -> 12V
- IC2 pad 26: /MCU/12V -> 12V
- IC2 pad 28: /MCU/GND -> GND
- IC2 pad 37: /MCU/5V -> 5V
- IC2 pad 38: /MCU/GND -> GND
- IC2 pad 4: /MCU/GND -> GND
- IC2 pad 6: /MCU/GND -> GND
- IC2 pad 7: /MCU/5V -> 5V
- IC3 pad 1: /MCU/GND -> GND
- IC3 pad 13: /MCU/GND -> GND
- IC3 pad 18: /MCU/GND -> GND
- IC3 pad 21: /MCU/5V -> 5V
- IC3 pad 25: /MCU/12V -> 12V
- IC3 pad 27: /MCU/GND -> GND
- IC3 pad 37: /MCU/5V -> 5V
- IC3 pad 38: /MCU/GND -> GND
- IC3 pad 4: /MCU/GND -> GND
- IC3 pad 7: /MCU/GND -> GND
- IC3 pad 8: /MCU/5V -> 5V
- R2 pad 2: /UART/GND -> GND
- SG pad : /MCU/5V -> 5V
Routing:
- net GND: track 0.00 -> 101.6 mm, vias 0 -> 12
- net 5V: track 0.00 -> 54.0 mm, vias 0 -> 6
- net /MCU/5V: track 52.5 -> 0.00 mm, vias 6 -> 0
- net LED_C15: track 31.1 -> 80.5 mm, vias 1 -> 4
- net LED_C12: track 39.5 -> 88.6 mm
- net LED_C8: track 25.1 -> 73.7 mm
- net LED_C9: track 22.3 -> 68.5 mm
- net LED_C13: track 36.3 -> 74.6 mm
- net 12V: track 0.00 -> 26.4 mm, vias 0 -> 1
- net /MCU/12V: track 26.4 -> 0.00 mm, vias 1 -> 0
- net LED_C14: track 41.3 -> 61.8 mm, vias 1 -> 2
- net LED_L0: track 23.4 -> 24.6 mm
- net /MCU/GND: vias 1 -> 0
- added copper zone on B.Cu, net GND
- added copper zone on F.Cu, net GND
Other:
- net class Default: clearance 0.2 -> 0.16
- net class Power: clearance 0.2 -> 1.6
- rule trace_clearance: 0.2 -> 0.16

Commit message: work in progress
Parts:
- added SG: 1.0, spark_gap_pad_1.0, B.Cu at (151.0, 123.1)
- added SG: 1.0, spark_gap_pad_1.0, B.Cu at (139.9, 117.7)
- added SG: 1.0, spark_gap_pad_1.0, B.Cu at (139.9, 119.7)
- added SG: 1.0, spark_gap_pad_1.0, B.Cu at (138.9, 119.7)
- added SG: 1.0, spark_gap_pad_1.0, B.Cu at (139.9, 118.7)
- added SG: 1.0, spark_gap_pad_1.0, B.Cu at (138.9, 118.7)
- added SG: 1.0, spark_gap_pad_1.0, B.Cu at (150.0, 121.1)
- added SG: 1.0, spark_gap_pad_1.0, B.Cu at (151.0, 124.1)
- added SG: 1.0, spark_gap_pad_1.0, B.Cu at (139.9, 120.7)
- added SG: 1.0, spark_gap_pad_1.0, B.Cu at (151.0, 122.1)
- added SG: 1.0, spark_gap_pad_1.0, B.Cu at (150.0, 122.1)
- added SG: 1.0, spark_gap_pad_1.0, B.Cu at (139.9, 121.7)
- added SG: 1.0, spark_gap_pad_1.0, B.Cu at (140.9, 121.7)
- C1, C2, C3, C4, C5, D2, FB1, R1: moved to B.Cu
- moved R3 30.1 mm to (154.3, 117.7), turned to 270 degrees
- moved C2 28.6 mm to (144.0, 114.1), turned to 270 degrees
- moved C3 28.1 mm to (146.0, 114.1), turned to 270 degrees
- moved R2 26.7 mm to (152.4, 117.7)
- moved C4 26.0 mm to (137.3, 117.7), turned to 90 degrees
- moved D2 21.2 mm to (157.0, 119.1), turned to 90 degrees
- moved FB1 14.6 mm to (153.7, 121.4), turned to 0 degrees
- moved R1 14.2 mm to (136.5, 123.4), turned to 180 degrees
- moved C5 13.3 mm to (153.7, 123.5)
- moved C1 8.38 mm to (151.9, 128.3), turned to 180 degrees
- moved D_RXTX1 5.01 mm to (136.8, 128.5), turned to 180 degrees
- moved IC1 2.60 mm to (145.1, 122.0)
- moved SG 0.40 mm to (141.4, 114.7)
- moved SG 0.40 mm to (141.4, 113.7)
- moved SG 0.40 mm to (148.6, 114.7)
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Connections:
- CON1 pad 6: (no net) -> N-0000076
- CON1 pad 7: (no net) -> N-0000079
- CON1 pad 8: (no net) -> N-0000078
- CON1 pad 9: (no net) -> N-0000077
Routing:
- net 5V: track 54.0 -> 101.7 mm, vias 6 -> 9
- net UART_RXD: track 25.7 -> 57.1 mm, vias 1 -> 2
- net UART_TXD: track 27.5 -> 50.1 mm, vias 1 -> 2
- net GND: track 101.6 -> 118.5 mm, vias 12 -> 13
- net 12V: track 26.4 -> 42.2 mm, vias 1 -> 3
- net N-0000080: track 0.00 -> 13.1 mm, vias 0 -> 1
- net N-0000069: track 0.00 -> 12.7 mm, vias 0 -> 2
- net /UART/USBD+: track 0.00 -> 8.99 mm, vias 0 -> 1
- net /UART/USBD-: track 0.00 -> 8.06 mm, vias 0 -> 1
- net LED_C4: track 41.0 -> 48.4 mm
- net N-0000073: track 0.00 -> 6.16 mm
- net N-0000057: track 0.00 -> 5.86 mm, vias 0 -> 1
- net N-0000066: track 0.00 -> 5.67 mm
- net N-0000081: track 0.00 -> 5.46 mm
- net LED_C5: track 24.6 -> 26.2 mm
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Other:
- net class Power: clearance 1.6 -> 0.16
- board text added: "C"
- board text added: "M"
- board text added: "agni"
- board text added: "ube"

Commit message: work in progress
Parts:
- added G***: LOGO, Logo_silk_polarity_external_5x1.4mm, F.Cu at (168.0, 93.0)
- added G***: LOGO, Logo_silk_CC-BY-SA_10x4.5mm, B.Cu at (160.0, 95.0)
- HOLE 3.4: value VAL** -> NE
- HOLE 3.4: value VAL** -> SW
- HOLE 3.4: value VAL** -> SE
- HOLE 3.4: value VAL** -> NW
Other:
- board text added: "2016"
- board text added: "5-12V"
- board text added: "C0"
- board text added: "C1"
- board text added: "C10"
- board text added: "C11"
- board text added: "C12"
- board text added: "C13"
- board text added: "C14"
- board text added: "C15"
- board text added: "C2"
- board text added: "C3"
- board text added: "C4"
- board text added: "C5"
- board text added: "C6"
- board text added: "C7"
- board text added: "C8"
- board text added: "C9"
- board text added: "Dirk Heisswolf"
- board text added: "L0"
- board text added: "L1"
- board text added: "L2"
- board text added: "L3"
- board text added: "RX"
- board text added: "RevA"
- board text added: "S12VR64"
- board text added: "S12VRP64"
- board text added: "TX"
- board text added: "http://hotwolf.github.io/MagniCube"
