File: Hardware/RevA/KiCad/MagniCube-RevA.kicad_pcb (KiCad board)
At the start: 2 copper layers, 50 x 50 mm, 136 parts, among them CON1 USB-MINI-B, CON2 DC_JACK, CON3 BDM, IC1 FT232RL, IC2 MC9S12VR64, IC3 MC9S12VRP64

Commit message: work in progress
Parts:
- IC3: value MC9S12VRP64 -> MC9S12XXXXX
- moved D2 1.15 mm to (157.0, 118.0)
- moved D1 0.22 mm to (153.6, 105.2)
- moved C1 0.10 mm to (151.9, 128.4)
- moved D_RXTX1 0.10 mm to (136.8, 128.4)
Routing:
- net GND: track 118.5 -> 494.6 mm, vias 13 -> 128
- net LED_C8: track 74.9 -> 76.8 mm
- net (no net): track 0.00 -> 1.73 mm
- net LED_C10: track 28.3 -> 29.2 mm
- net 12V: track 42.2 -> 41.6 mm
Other:
- board text removed: "S12VR64"
- board text removed: "S12VRP64"

Commit message: work in progress
Parts:
- moved G*** 0.92 mm to (168.6, 92.3), turned to 90 degrees
Routing:
- net GND: track 494.6 -> 629.7 mm, vias 128 -> 163
- net 5V: track 101.7 -> 104.6 mm
- net (no net): track 1.73 -> 0.00 mm
- net LED_C1: track 29.5 -> 28.7 mm
- net LED_C0: track 43.3 -> 42.5 mm
- net LED_L0: track 24.6 -> 24.1 mm
