File: Hardware/RevA/KiCad/MagniCube-RevA-MCU.sch (KiCad schematic (older format))
At the start: 11 parts, among them CON1 BDM, IC1a MC9S12VR64, IC1b MC9S12VRP64

Commit message: schematic in progress
Parts:
- added CON1: DC_JACK, symbol DC_JACK
- C1a1: renamed from C1a; value C -> 4.7uF
- C1b1: renamed from C1b; value C -> 4.7uF
- C2a1: renamed from C2a; value C -> 100nf
- C2b1: renamed from C2b; value C -> 100nf
- C3a1: renamed from C3a; value C -> 100nf
- C3b1: renamed from C3b; value C -> 100nf
- renumbered C4a to C4a1, C4b to C4b1, CON1 to CON2, IC1a to IC1a1, IC1b to IC1b1
Connections:
- net labels added: VIO, VSUP
- net labels removed: 12V, 5V
- wire segments 119 -> 125

Commit message: PCB in progress
Parts:
- renumbered C1b1 to C10, C2b1 to C11, C3b1 to C12, C4b1 to C13, C1a1 to C6, C2a1 to C7, C3a1 to C8, C4a1 to C9, CON1 to CON2, CON2 to CON3, IC1a1 to IC2, IC1b1 to IC3
Changed lines of the file:
@@
 Sheet 3 4
 Title "MCU"
-Date "14 apr 2016"
+Date "18 apr 2016"
 Rev "RevA"
 Comp "Dirk Heisswolf"
@@
 $EndDescr
 $Comp
-L BDM CON2
+L BDM CON3
 U 1 1 544FF341
 P 2800 4300
-F 0 "CON2" H 2800 3950 60  0000 C CNN
+F 0 "CON3" H 2800 3950 60  0000 C CNN
 F 1 "BDM" H 2800 4700 60  0000 C CNN
 F 2 "~" H 3350 3600 60  0000 C CNN
@@
 UART_TXD
 $Comp
-L MC9S12VR64 IC1a1
+L MC9S12VR64 IC2
 U 1 1 57040B96
 P 3350 2400
-F 0 "IC1a1" H 3350 2500 60  0000 C CNN
+F 0 "IC2" H 3350 2500 60  0000 C CNN
 F 1 "MC9S12VR64" H 3350 2300 60  0000 C CNN
 F 2 "~" H 3900 2300 60  0000 C CNN
@@
 $EndComp
 $Comp
-L MC9S12VRP64 IC1b1
+L MC9S12VRP64 IC3
 U 1 1 57040BB9
 P 6150 2400
-F 0 "IC1b1" H 6150 2500 60  0000 C CNN
+F 0 "IC3" H 6150 2500 60  0000 C CNN
 F 1 "MC9S12VRP64" H 6150 2300 60  0000 C CNN
 F 2 "~" H 6700 2300 60  0000 C CNN
@@
 BKGD
 $Comp
-L C C1b1
+L C C10
 U 1 1 57043AE1
 P 800 2300
-F 0 "C1b1" H 800 2400 40  0000 L CNN
+F 0 "C10" H 800 2400 40  0000 L CNN
 F 1 "4.7uF" H 806 2215 40  0000 L CNN
 F 2 "~" H 838 2150 30  0000 C CNN
@@
 $EndComp
 $Comp
-L C C2b1
+L C C11
 U 1 1 57043AF0
 P 1050 2300
-F 0 "C2b1" H 1050 2400 40  0000 L CNN
+F 0 "C11" H 1050 2400 40  0000 L CNN
 F 1 "100nf" H 1056 2215 40  0000 L CNN
 F 2 "~" H 1088 2150 30  0000 C CNN
@@
 $EndComp
 $Comp
-L C C3b1
+L C C12
 U 1 1 57043AFD
 P 1300 2300
-F 0 "C3b1" H 1300 2400 40  0000 L CNN
+F 0 "C12" H 1300 2400 40  0000 L CNN
 F 1 "100nf" H 1306 2215 40  0000 L CNN
 F 2 "~" H 1338 2150 30  0000 C CNN
@@
 $EndComp
 $Comp
-L C C4b1
+L C C13
 U 1 1 57044866
 P 1650 2300
-F 0 "C4b1" H 1650 2400 40  0000 L CNN
+F 0 "C13" H 1650 2400 40  0000 L CNN
 F 1 "C" H 1656 2215 40  0000 L CNN
 F 2 "~" H 1688 2150 30  0000 C CNN
@@
 $EndComp
 $Comp
-L C C1a1
+L C C6
 U 1 1 57044C68
 P 800 1400
-F 0 "C1a1" H 800 1500 40  0000 L CNN
+F 0 "C6" H 800 1500 40  0000 L CNN
 F 1 "4.7uF" H 806 1315 40  0000 L CNN
 F 2 "~" H 838 1250 30  0000 C CNN
@@
 $EndComp
 $Comp
-L C C2a1
+L C C7
 U 1 1 57044C6E
 P 1050 1400
-F 0 "C2a1" H 1050 1500 40  0000 L CNN
+F 0 "C7" H 1050 1500 40  0000 L CNN
 F 1 "100nf" H 1056 1315 40  0000 L CNN
 F 2 "~" H 1088 1250 30  0000 C CNN
@@
 $EndComp
 $Comp
-L C C3a1
+L C C8
 U 1 1 57044C74
 P 1300 1400
-F 0 "C3a1" H 1300 1500 40  0000 L CNN
+F 0 "C8" H 1300 1500 40  0000 L CNN
 F 1 "100nf" H 1306 1315 40  0000 L CNN
 F 2 "~" H 1338 1250 30  0000 C CNN
@@
 $EndComp
 $Comp
-L C C4a1
+L C C9
 U 1 1 57044C80
 P 1650 1400
-F 0 "C4a1" H 1650 1500 40  0000 L CNN
+F 0 "C9" H 1650 1500 40  0000 L CNN
 F 1 "C" H 1656 1315 40  0000 L CNN
 F 2 "~" H 1688 1250 30  0000 C CNN
@@
 $EndComp
 $Comp
-L DC_JACK CON1
+L DC_JACK CON2
 U 1 1 570D05EC
 P 950 3200
-F 0 "CON1" H 950 3350 60  0000 C CNN
+F 0 "CON2" H 950 3350 60  0000 C CNN
 F 1 "DC_JACK" H 950 3050 60  0000 C CNN
 F 2 "" H 950 3200 60  0000 C CNN

Commit message: work in progress
Parts:
- removed C12: 100nf, ~, symbol C
- removed C13, C9: C, ~, symbol C
- C10: value 4.7uF -> 100nf
Connections:
- wire segments 125 -> 121
Other:
- moved on the sheet: C10, C11
Changed lines of the file:
@@
 Sheet 3 4
 Title "MCU"
-Date "18 apr 2016"
+Date "19 apr 2016"
 Rev "RevA"
 Comp "Dirk Heisswolf"
@@
 $EndComp
 $Comp
-L GND #PWR_GND07
+L GND #PWR?
 U 1 1 57042C33
 P 4550 2700
-F 0 "#PWR_GND07" H 4550 2700 30  0001 C CNN
+F 0 "#PWR?" H 4550 2700 30  0001 C CNN
 F 1 "GND" H 4550 2630 30  0001 C CNN
 F 2 "~" H 4550 2700 60  0000 C CNN
@@
 $EndComp
 $Comp
-L 12V #PWR_SUPPLY4
-U 1 1 57042D02
-P 1650 2050
-F 0 "#PWR_SUPPLY4" H 1650 2150 40  0001 C CNN
-F 1 "VSUP" H 1650 2199 40  0000 C CNN
-F 2 "~" H 1650 2050 60  0000 C CNN
-F 3 "~" H 1650 2050 60  0000 C CNN
-	1    1650 2050
-	1    0    0    -1
-$EndComp
-$Comp
-L GND #PWR08
+L GND #PWR?
 U 1 1 57042D65
 P 2800 3550
-F 0 "#PWR08" H 2800 3550 30  0001 C CNN
+F 0 "#PWR?" H 2800 3550 30  0001 C CNN
 F 1 "GND" H 2800 3480 30  0001 C CNN
 F 2 "~" H 2800 3550 60  0000 C CNN
@@
 $EndComp
 $Comp
-L GND #PWR09
+L GND #PWR?
 U 1 1 57042D6B
 P 3300 3550
-F 0 "#PWR09" H 3300 3550 30  0001 C CNN
+F 0 "#PWR?" H 3300 3550 30  0001 C CNN
 F 1 "GND" H 3300 3480 30  0001 C CNN
 F 2 "~" H 3300 3550 60  0000 C CNN
@@
 $EndComp
 $Comp
-L GND #PWR010
+L GND #PWR?
 U 1 1 57042D85
 P 5600 3550
-F 0 "#PWR010" H 5600 3550 30  0001 C CNN
+F 0 "#PWR?" H 5600 3550 30  0001 C CNN
 F 1 "GND" H 5600 3480 30  0001 C CNN
 F 2 "~" H 5600 3550 60  0000 C CNN
@@
 $EndComp
 $Comp
-L GND #PWR011
+L GND #PWR?
 U 1 1 57042D8B
 P 6100 3550
-F 0 "#PWR011" H 6100 3550 30  0001 C CNN
+F 0 "#PWR?" H 6100 3550 30  0001 C CNN
 F 1 "GND" H 6100 3480 30  0001 C CNN
 F 2 "~" H 6100 3550 60  0000 C CNN
@@
 $EndComp
 $Comp
-L GND #PWR_GND012
+L GND #PWR?
 U 1 1 57042F3F
 P 7350 2800
-F 0 "#PWR_GND012" H 7350 2800 30  0001 C CNN
+F 0 "#PWR?" H 7350 2800 30  0001 C CNN
 F 1 "GND" H 7350 2730 30  0001 C CNN
 F 2 "~" H 7350 2800 60  0000 C CNN
@@
 $EndComp
 $Comp
-L GND #PWR_GND013
-U 1 1 57043099
-P 800 2550
-F 0 "#PWR_GND013" H 800 2550 30  0001 C CNN
-F 1 "GND" H 800 2480 30  0001 C CNN
-F 2 "~" H 800 2550 60  0000 C CNN
-F 3 "~" H 800 2550 60  0000 C CNN
-	1    800  2550
-	1    0    0    -1
-$EndComp
-$Comp
-L GND #PWR_GND014
+L GND #PWR?
 U 1 1 5704309F
 P 3900 1150
-F 0 "#PWR_GND014" H 3900 1150 30  0001 C CNN
+F 0 "#PWR?" H 3900 1150 30  0001 C CNN
 F 1 "GND" H 3900 1080 30  0001 C CNN
 F 2 "~" H 3900 1150 60  0000 C CNN
@@
 $EndComp
 $Comp
-L GND #PWR_GND015
+L GND #PWR?
 U 1 1 5704344E
 P 6700 1150
-F 0 "#PWR_GND015" H 6700 1150 30  0001 C CNN
+F 0 "#PWR?" H 6700 1150 30  0001 C CNN
 F 1 "GND" H 6700 1080 30  0001 C CNN
 F 2 "~" H 6700 1150 60  0000 C CNN
@@
 $EndComp
 $Comp
-L GND #PWR_GND016
+L GND #PWR?
 U 1 1 57043622
 P 3400 4500
-F 0 "#PWR_GND016" H 3400 4500 30  0001 C CNN
+F 0 "#PWR?" H 3400 4500 30  0001 C CNN
 F 1 "GND" H 3400 4430 30  0001 C CNN
 F 2 "~" H 3400 4500 60  0000 C CNN
@@
 L C C10
 U 1 1 57043AE1
-P 800 2300
-F 0 "C10" H 800 2400 40  0000 L CNN
-F 1 "4.7uF" H 806 2215 40  0000 L CNN
-F 2 "~" H 838 2150 30  0000 C CNN
-F 3 "~" H 800 2300 60  0000 C CNN
-	1    800  2300
+P 1550 1400
+F 0 "C10" H 1550 1500 40  0000 L CNN
+F 1 "100nf" H 1556 1315 40  0000 L CNN
+F 2 "~" H 1588 1250 30  0000 C CNN
+F 3 "~" H 1550 1400 60  0000 C CNN
+	1    1550 1400
 	1    0    0    -1
 $EndComp
@@
 L C C11
 U 1 1 57043AF0
-P 1050 2300
-F 0 "C11" H 1050 2400 40  0000 L CNN
-F 1 "100nf" H 1056 2215 40  0000 L CNN
-F 2 "~" H 1088 2150 30  0000 C CNN
-F 3 "~" H 1050 2300 60  0000 C CNN
-	1    1050 2300
-	1    0    0    -1
-$EndComp
-$Comp
-L C C12
-U 1 1 57043AFD
-P 1300 2300
-F 0 "C12" H 1300 2400 40  0000 L CNN
-F 1 "100nf" H 1306 2215 40  0000 L CNN
-F 2 "~" H 1338 2150 30  0000 C CNN
-F 3 "~" H 1300 2300 60  0000 C CNN
-	1    1300 2300
-	1    0    0    -1
-$EndComp
-$Comp
-L 5V #PWR_IO5
-U 1 1 5704482E
-P 800 2050
-F 0 "#PWR_IO5" H 800 2150 40  0001 C CNN
-F 1 "VIO" H 800 2199 40  0000 C CNN
-F 2 "~" H 800 2050 60  0000 C CNN
-F 3 "~" H 800 2050 60  0000 C CNN
-	1    800  2050
-	1    0    0    -1
-$EndComp
-$Comp
-L C C13
-U 1 1 57044866
-P 1650 2300
-F 0 "C13" H 1650 2400 40  0000 L CNN
-F 1 "C" H 1656 2215 40  0000 L CNN
-F 2 "~" H 1688 2150 30  0000 C CNN
-F 3 "~" H 1650 2300 60  0000 C CNN
-	1    1650 2300
-	1    0    0    -1
-$EndComp
-$Comp
-L 12V #PWR_SUPPLY3
-U 1 1 57044C5C
-P 1650 1150
-F 0 "#PWR_SUPPLY3" H 1650 1250 40  0001 C CNN
-F 1 "VSUP" H 1650 1299 40  0000 C CNN
-F 2 "~" H 1650 1150 60  0000 C CNN
-F 3 "~" H 1650 1150 60  0000 C CNN
-	1    1650 1150
-	1    0    0    -1
-$EndComp
-$Comp
-L GND #PWR_GND017
+P 1800 1400
+F 0 "C11" H 1800 1500 40  0000 L CNN
+F 1 "100nf" H 1806 1315 40  0000 L CNN
+F 2 "~" H 1838 1250 30  0000 C CNN
+F 3 "~" H 1800 1400 60  0000 C CNN
+	1    1800 1400
+	1    0    0    -1
+$EndComp
+$Comp
+L GND #PWR?
 U 1 1 57044C62
 P 800 1650
-F 0 "#PWR_GND017" H 800 1650 30  0001 C CNN
+F 0 "#PWR?" H 800 1650 30  0001 C CNN
 F 1 "GND" H 800 1580 30  0001 C CNN
 F 2 "~" H 800 1650 60  0000 C CNN
@@
 F 3 "~" H 800 1150 60  0000 C CNN
 	1    800  1150
-	1    0    0    -1
-$EndComp
-$Comp
-L C C9
-U 1 1 57044C80
-P 1650 1400
-F 0 "C9" H 1650 1500 40  0000 L CNN
-F 1 "C" H 1656 1315 40  0000 L CNN
-F 2 "~" H 1688 1250 30  0000 C CNN
-F 3 "~" H 1650 1400 60  0000 C CNN
-	1    1650 1400
 	1    0    0    -1
 $EndComp
@@
 $EndComp
 $Comp
-L GND #PWR_GND018
+L GND #PWR?
 U 1 1 570D075F
 P 1250 3300
-F 0 "#PWR_GND018" H 1250 3300 30  0001 C CNN
+F 0 "#PWR?" H 1250 3300 30  0001 C CNN
 F 1 "GND" H 1250 3230 30  0001 C CNN
 F 2 "~" H 1250 3300 60  0000 C CNN
@@
 	1    0    0    -1
 $EndComp
+Text Label 5700 3700 1    39   ~ 0
+RESET
+$Comp
+L GND #PWR?
+U 1 1 57160D4B
+P 2050 1950
+F 0 "#PWR?" H 2050 1950 30  0001 C CNN
+F 1 "GND" H 2050 1880 30  0001 C CNN
+F 2 "~" H 2050 1950 60  0000 C CNN
+F 3 "~" H 2050 1950 60  0000 C CNN
+	1    2050 1950
+	1    0    0    -1
+$EndComp
+$Comp
+L GND #PWR?
+U 1 1 57160D51
+P 4850 1950
+F 0 "#PWR?" H 4850 1950 30  0001 C CNN
+F 1 "GND" H 4850 1880 30  0001 C CNN
+F 2 "~" H 4850 1950 60  0000 C CNN
+F 3 "~" H 4850 1950 60  0000 C CNN
+	1    4850 1950
+	1    0    0    -1
+$EndComp
 Wire Bus Line
 	7550 1000 7550 3800
@@
 	2150 2150 2250 2150
 Wire Wire Line
-	2150 1850 2250 1850
+	2050 1850 2250 1850
 Connection ~ 2150 2150
 Wire Wire Line
@@
 	4950 2150 5050 2150
 Wire Wire Line
-	4950 1850 5050 1850
+	4850 1850 5050 1850
 Connection ~ 4950 2150
 Wire Wire Line
@@
 	6400 3650 6400 3500
 Wire Wire Line
-	3800 1300 3800 1100
-Wire Wire Line
-	3800 1100 3900 1100
-Wire Wire Line
-	3900 1100 3900 1150
-Wire Wire Line
 	3900 1300 4050 1300
 Wire Wire Line
@@
 	2100 4450 2200 4450
 Wire Wire Line
-	800  2100 1300 2100
-Connection ~ 1050 2100
-Wire Wire Line
-	800  2500 1650 2500
-Connection ~ 1050 2500
-Connection ~ 1300 2500
-Wire Wire Line
-	1650 2050 1650 2100
-Wire Wire Line
-	800  2050 800  2100
-Wire Wire Line
-	800  2500 800  2550
-Wire Wire Line
-	800  1200 1300 1200
+	800  1200 1800 1200
 Connection ~ 1050 1200
-Wire Wire Line
-	800  1600 1650 1600
 Connection ~ 1050 1600
 Connection ~ 1300 1600
 Wire Wire Line
-	1650 1150 1650 1200
-Wire Wire Line
 	800  1150 800  1200
 Wire Wire Line
@@
 Wire Wire Line
 	1100 3200 1100 3250
-Text Label 5700 3700 1    39   ~ 0
-RESET
+Wire Wire Line
+	4850 1950 4850 1850
+Connection ~ 4950 1850
+Wire Wire Line
+	2050 1950 2050 1850
+Connection ~ 2150 1850
+Connection ~ 1300 1200
+Connection ~ 1550 1200
+Wire Wire Line
+	800  1600 1800 1600
+Connection ~ 1550 1600
+Wire Wire Line
+	3800 1300 3800 1100
+Wire Wire Line
+	3800 1100 3900 1100
+Wire Wire Line
+	3900 1100 3900 1150
 $EndSCHEMATC

Commit message: work in progress
Connections:
- net labels added: 12V, 5V
- net labels removed: VSUP
- wire segments 121 -> 128

Commit message: work in progress
Parts:
- added D1: SCHOTTKY, ~, symbol SCHOTTKY
Connections:
- net labels removed: VIO
- wire segments 128 -> 129

Commit message: work in progress
Parts:
- added C11: 100nf, ~, symbol C
- renumbered C11 to C10, C10 to C9
Changed lines of the file:
@@
 EESchema Schematic File Version 2
 LIBS:MagniCube
-LIBS:w_connectors
-LIBS:w_device
 LIBS:MagniCube-RevA-cache
 EELAYER 27 0
@@
 Sheet 3 4
 Title "MCU"
-Date "21 apr 2016"
+Date "22 apr 2016"
 Rev "RevA"
 Comp "Dirk Heisswolf"
@@
 BKGD
 $Comp
-L C C10
+L C C9
 U 1 1 57043AE1
 P 1550 1400
-F 0 "C10" H 1550 1500 40  0000 L CNN
+F 0 "C9" H 1550 1500 40  0000 L CNN
 F 1 "100nf" H 1556 1315 40  0000 L CNN
 F 2 "~" H 1588 1250 30  0000 C CNN
@@
 $EndComp
 $Comp
-L C C11
+L C C10
 U 1 1 57043AF0
 P 1800 1400
-F 0 "C11" H 1800 1500 40  0000 L CNN
+F 0 "C10" H 1800 1500 40  0000 L CNN
 F 1 "100nf" H 1806 1315 40  0000 L CNN
 F 2 "~" H 1838 1250 30  0000 C CNN
@@
 Text Label 3400 4450 2    39   ~ 0
 GND
-Text Label 1800 1600 2    39   ~ 0
+Text Label 2050 1600 2    39   ~ 0
 GND
 $Comp
@@
 	1    0    0    -1
 $EndComp
-Text Label 1800 1200 2    39   ~ 0
+Text Label 2050 1200 2    39   ~ 0
 5V
 $Comp
@@
 	2100 4450 2200 4450
 Wire Wire Line
-	800  1200 1800 1200
+	800  1200 2050 1200
 Connection ~ 1050 1200
 Connection ~ 1050 1600
@@
 Connection ~ 1550 1200
 Wire Wire Line
-	800  1600 1800 1600
+	800  1600 2050 1600
 Connection ~ 1550 1600
 Wire Wire Line
@@
 Wire Wire Line
 	1400 3250 1400 3300
+$Comp
+L C C11
+U 1 1 571A5894
+P 2050 1400
+F 0 "C11" H 2050 1500 40  0000 L CNN
+F 1 "100nf" H 2056 1315 40  0000 L CNN
+F 2 "~" H 2088 1250 30  0000 C CNN
+F 3 "~" H 2050 1400 60  0000 C CNN
+	1    2050 1400
+	1    0    0    -1
+$EndComp
+Connection ~ 1800 1200
+Connection ~ 1800 1600
 $EndSCHEMATC

Commit message: work in progress
Connections:
- wire segments 129 -> 132
Changed lines of the file:
@@
 Sheet 3 4
 Title "MCU"
-Date "22 apr 2016"
+Date "23 apr 2016"
 Rev "RevA"
 Comp "Dirk Heisswolf"
@@
 Text GLabel 7050 4200 3    39   Input ~ 0
 UART_TXD
-$Comp
-L MC9S12VR64 IC2
-U 1 1 57040B96
-P 3350 2400
-F 0 "IC2" H 3350 2500 60  0000 C CNN
-F 1 "MC9S12VR64" H 3350 2300 60  0000 C CNN
-F 2 "~" H 3900 2300 60  0000 C CNN
-F 3 "~" H 3900 2300 60  0000 C CNN
-	1    3350 2400
-	1    0    0    -1
-$EndComp
 $Comp
 L MC9S12VRP64 IC3
@@
 NoConn ~ 2250 2850
 $Comp
-L GND #PWR07
+L GND #PWR011
 U 1 1 57042C33
 P 4550 2700
-F 0 "#PWR07" H 4550 2700 30  0001 C CNN
+F 0 "#PWR011" H 4550 2700 30  0001 C CNN
 F 1 "GND" H 4550 2630 30  0001 C CNN
 F 2 "~" H 4550 2700 60  0000 C CNN
@@
 $EndComp
 $Comp
-L GND #PWR08
+L GND #PWR012
 U 1 1 57042D65
 P 2800 3700
-F 0 "#PWR08" H 2800 3700 30  0001 C CNN
+F 0 "#PWR012" H 2800 3700 30  0001 C CNN
 F 1 "GND" H 2800 3630 30  0001 C CNN
 F 2 "~" H 2800 3700 60  0000 C CNN
@@
 $EndComp
 $Comp
-L GND #PWR09
+L GND #PWR013
 U 1 1 57042D6B
 P 3300 3700
-F 0 "#PWR09" H 3300 3700 30  0001 C CNN
+F 0 "#PWR013" H 3300 3700 30  0001 C CNN
 F 1 "GND" H 3300 3630 30  0001 C CNN
 F 2 "~" H 3300 3700 60  0000 C CNN
@@
 $EndComp
 $Comp
-L GND #PWR010
+L GND #PWR014
 U 1 1 57042D85
 P 5600 3700
-F 0 "#PWR010" H 5600 3700 30  0001 C CNN
+F 0 "#PWR014" H 5600 3700 30  0001 C CNN
 F 1 "GND" H 5600 3630 30  0001 C CNN
 F 2 "~" H 5600 3700 60  0000 C CNN
@@
 $EndComp
 $Comp
-L GND #PWR011
+L GND #PWR015
 U 1 1 57042D8B
 P 6100 3700
-F 0 "#PWR011" H 6100 3700 30  0001 C CNN
+F 0 "#PWR015" H 6100 3700 30  0001 C CNN
 F 1 "GND" H 6100 3630 30  0001 C CNN
 F 2 "~" H 6100 3700 60  0000 C CNN
@@
 $EndComp
 $Comp
-L GND #PWR012
+L GND #PWR016
 U 1 1 57042F3F
 P 7350 2800
-F 0 "#PWR012" H 7350 2800 30  0001 C CNN
+F 0 "#PWR016" H 7350 2800 30  0001 C CNN
 F 1 "GND" H 7350 2730 30  0001 C CNN
 F 2 "~" H 7350 2800 60  0000 C CNN
@@
 $EndComp
 $Comp
-L GND #PWR013
+L GND #PWR017
 U 1 1 5704309F
 P 3900 1150
-F 0 "#PWR013" H 3900 1150 30  0001 C CNN
+F 0 "#PWR017" H 3900 1150 30  0001 C CNN
 F 1 "GND" H 3900 1080 30  0001 C CNN
 F 2 "~" H 3900 1150 60  0000 C CNN
@@
 $EndComp
 $Comp
-L GND #PWR014
+L GND #PWR018
 U 1 1 5704344E
 P 6700 1150
-F 0 "#PWR014" H 6700 1150 30  0001 C CNN
+F 0 "#PWR018" H 6700 1150 30  0001 C CNN
 F 1 "GND" H 6700 1080 30  0001 C CNN
 F 2 "~" H 6700 1150 60  0000 C CNN
@@
 $EndComp
 $Comp
-L GND #PWR015
+L GND #PWR019
 U 1 1 57043622
 P 3400 4500
-F 0 "#PWR015" H 3400 4500 30  0001 C CNN
+F 0 "#PWR019" H 3400 4500 30  0001 C CNN
 F 1 "GND" H 3400 4430 30  0001 C CNN
 F 2 "~" H 3400 4500 60  0000 C CNN
@@
 $EndComp
 $Comp
-L GND #PWR016
+L GND #PWR020
 U 1 1 57044C62
 P 800 1650
-F 0 "#PWR016" H 800 1650 30  0001 C CNN
+F 0 "#PWR020" H 800 1650 30  0001 C CNN
 F 1 "GND" H 800 1580 30  0001 C CNN
 F 2 "~" H 800 1650 60  0000 C CNN
@@
 $EndComp
 $Comp
-L GND #PWR017
+L GND #PWR021
 U 1 1 570D075F
 P 1400 3300
-F 0 "#PWR017" H 1400 3300 30  0001 C CNN
+F 0 "#PWR021" H 1400 3300 30  0001 C CNN
 F 1 "GND" H 1400 3230 30  0001 C CNN
 F 2 "~" H 1400 3300 60  0000 C CNN
@@
 RESET
 $Comp
-L GND #PWR018
+L GND #PWR022
 U 1 1 57160D4B
 P 2050 1950
-F 0 "#PWR018" H 2050 1950 30  0001 C CNN
+F 0 "#PWR022" H 2050 1950 30  0001 C CNN
 F 1 "GND" H 2050 1880 30  0001 C CNN
 F 2 "~" H 2050 1950 60  0000 C CNN
@@
 $EndComp
 $Comp
-L GND #PWR019
+L GND #PWR023
 U 1 1 57160D51
 P 4850 1950
-F 0 "#PWR019" H 4850 1950 30  0001 C CNN
+F 0 "#PWR023" H 4850 1950 30  0001 C CNN
 F 1 "GND" H 4850 1880 30  0001 C CNN
 F 2 "~" H 4850 1950 60  0000 C CNN
@@
 	1    0    0    -1
 $EndComp
-Text Label 3800 1300 1    39   ~ 0
-GND
-Text Label 6600 1300 1    39   ~ 0
-GND
-Text Label 2150 2150 1    39   ~ 0
-GND
-Text Label 4950 2150 1    39   ~ 0
-GND
-Text Label 3300 3700 1    39   ~ 0
-GND
-Text Label 2800 3700 1    39   ~ 0
-GND
-Text Label 1400 3250 2    39   ~ 0
-GND
-Text Label 7250 2750 0    39   ~ 0
-GND
-Text Label 3400 4450 2    39   ~ 0
-GND
-Text Label 2050 1600 2    39   ~ 0
-GND
-$Comp
-L 12V #PWR25
+$Comp
+L 12V #PWR024
 U 1 1 57180AB5
 P 4650 2900
-F 0 "#PWR25" H 4650 3000 40  0001 C CNN
+F 0 "#PWR024" H 4650 3000 40  0001 C CNN
 F 1 "12V" H 4650 3049 40  0000 C CNN
 F 2 "~" H 4650 2900 60  0000 C CNN
@@
 $EndComp
 $Comp
-L 12V #PWR34
+L 12V #PWR025
 U 1 1 57180AC9
 P 7450 2900
-F 0 "#PWR34" H 7450 3000 40  0001 C CNN
+F 0 "#PWR025" H 7450 3000 40  0001 C CNN
 F 1 "12V" H 7450 3049 40  0000 C CNN
 F 2 "~" H 7450 2900 60  0000 C CNN
@@
 	1    0    0    -1
 $EndComp
-Text Label 4450 2650 0    39   ~ 0
-GND
-Text Label 1400 3150 2    39   ~ 0
-12V
-Text Label 4500 2950 0    39   ~ 0
-12V
-Text Label 7300 2950 0    39   ~ 0
-12V
-$Comp
-L 12V #PWR13
+$Comp
+L 12V #PWR026
 U 1 1 57180C44
 P 1400 3100
-F 0 "#PWR13" H 1400 3200 40  0001 C CNN
+F 0 "#PWR026" H 1400 3200 40  0001 C CNN
 F 1 "12V" H 1400 3249 40  0000 C CNN
 F 2 "~" H 1400 3100 60  0000 C CNN
@@
 $EndComp
 $Comp
-L 5V #PWR11
+L 5V #PWR027
 U 1 1 57180E29
 P 800 1150
-F 0 "#PWR11" H 800 1250 40  0001 C CNN
+F 0 "#PWR027" H 800 1250 40  0001 C CNN
 F 1 "5V" H 800 1299 40  0000 C CNN
 F 2 "~" H 800 1150 60  0000 C CNN
@@
 	1    0    0    -1
 $EndComp
-Text Label 2050 1200 2    39   ~ 0
-5V
-$Comp
-L 5V #PWR23
+$Comp
+L 5V #PWR028
 U 1 1 57180ED2
 P 4050 1250
-F 0 "#PWR23" H 4050 1350 40  0001 C CNN
+F 0 "#PWR028" H 4050 1350 40  0001 C CNN
 F 1 "5V" H 4050 1399 40  0000 C CNN
 F 2 "~" H 4050 1250 60  0000 C CNN
@@
 	1    0    0    -1
 $EndComp
-Text Label 3900 1300 0    39   ~ 0
-5V
-$Comp
-L 5V #PWR32
+$Comp
+L 5V #PWR029
 U 1 1 57180F65
 P 6850 1250
-F 0 "#PWR32" H 6850 1350 40  0001 C CNN
+F 0 "#PWR029" H 6850 1350 40  0001 C CNN
 F 1 "5V" H 6850 1399 40  0000 C CNN
 F 2 "~" H 6850 1250 60  0000 C CNN
@@
 	1    0    0    -1
 $EndComp
-Text Label 6700 1300 0    39   ~ 0
-5V
-$Comp
-L 5V #PWR27
+$Comp
+L 5V #PWR030
 U 1 1 57180FF6
 P 4850 2500
-F 0 "#PWR27" H 4850 2600 40  0001 C CNN
+F 0 "#PWR030" H 4850 2600 40  0001 C CNN
 F 1 "5V" H 4850 2649 40  0000 C CNN
 F 2 "~" H 4850 2500 60  0000 C CNN
@@
 $EndComp
 $Comp
-L 5V #PWR16
+L 5V #PWR031
 U 1 1 57180FFC
 P 2050 2400
-F 0 "#PWR16" H 2050 2500 40  0001 C CNN
+F 0 "#PWR031" H 2050 2500 40  0001 C CNN
 F 1 "5V" H 2050 2549 40  0000 C CNN
 F 2 "~" H 2050 2400 60  0000 C CNN
@@
 	1    0    0    -1
 $EndComp
-Text Label 2250 2450 2    39   ~ 0
-5V
-Text Label 5050 2550 2    39   ~ 0
-5V
-Text Label 5600 3700 1    39   ~ 0
-GND
-Text Label 6100 3700 1    39   ~ 0
-GND
-$Comp
-L 5V #PWR21
+$Comp
+L 5V #PWR032
 U 1 1 5718116C
 P 3550 3650
-F 0 "#PWR21" H 3550 3750 40  0001 C CNN
+F 0 "#PWR032" H 3550 3750 40  0001 C CNN
 F 1 "5V" H 3550 3799 40  0000 C CNN
 F 2 "~" H 3550 3650 60  0000 C CNN
@@
 $EndComp
 $Comp
-L 5V #PWR30
+L 5V #PWR033
 U 1 1 57181172
 P 6350 3650
-F 0 "#PWR30" H 6350 3750 40  0001 C CNN
+F 0 "#PWR033" H 6350 3750 40  0001 C CNN
 F 1 "5V" H 6350 3799 40  0000 C CNN
 F 2 "~" H 6350 3650 60  0000 C CNN
@@
 	1    0    0    -1
 $EndComp
-Text Label 3600 3700 3    39   ~ 0
-5V
-Text Label 6400 3700 3    39   ~ 0
-5V
-Text Label 3400 4150 2    39   ~ 0
-5V
-$Comp
-L 5V #PWR19
+$Comp
+L 5V #PWR034
 U 1 1 5718E2B5
 P 3400 4100
-F 0 "#PWR19" H 3400 4200 40  0001 C CNN
+F 0 "#PWR034" H 3400 4200 40  0001 C CNN
 F 1 "5V" H 3400 4249 40  0000 C CNN
 F 2 "~" H 3400 4100 60  0000 C CNN
@@
 	5600 3700 5600 3500
 Wire Wire Line
-	4450 2850 4450 2950
-Wire Wire Line
 	7250 2750 7350 2750
 Wire Wire Line
@@
 Connection ~ 1800 1200
 Connection ~ 1800 1600
+$Comp
+L MC9S12VR64 IC2
+U 1 1 57040B96
+P 3350 2400
+F 0 "IC2" H 3350 2500 60  0000 C CNN
+F 1 "MC9S12VR64" H 3350 2300 60  0000 C CNN
+F 2 "~" H 3900 2300 60  0000 C CNN
+F 3 "~" H 3900 2300 60  0000 C CNN
+	1    3350 2400
+	1    0    0    -1
+$EndComp
+Text Label 7300 2950 0    39   ~ 0
+12V
+Wire Wire Line
+	4450 2950 4450 2850
+$Comp
+L PWR_FLAG #FLG035
+U 1 1 571AE389
+P 750 4950
+F 0 "#FLG035" H 750 5045 30  0001 C CNN
+F 1 "PWR_FLAG" H 750 5130 30  0000 C CNN
+F 2 "" H 750 4950 60  0000 C CNN
+F 3 "" H 750 4950 60  0000 C CNN
+	1    750  4950
+	-1   0    0    1
+$EndComp
+$Comp
+L PWR_FLAG #FLG036
+U 1 1 571AE398
+P 1000 4950
+F 0 "#FLG036" H 1000 5045 30  0001 C CNN
+F 1 "PWR_FLAG" H 1000 5130 30  0000 C CNN
+F 2 "" H 1000 4950 60  0000 C CNN
+F 3 "" H 1000 4950 60  0000 C CNN
+	1    1000 4950
+	-1   0    0    1
+$EndComp
+$Comp
+L PWR_FLAG #FLG037
+U 1 1 571AE3A7
+P 1250 5150
+F 0 "#FLG037" H 1250 5245 30  0001 C CNN
+F 1 "PWR_FLAG" H 1250 5330 30  0000 C CNN
+F 2 "" H 1250 5150 60  0000 C CNN
+F 3 "" H 1250 5150 60  0000 C CNN
+	1    1250 5150
+	1    0    0    -1
+$EndComp
+$Comp
+L 5V #PWR038
+U 1 1 571AE3B4
+P 1000 4900
+F 0 "#PWR038" H 1000 5000 40  0001 C CNN
+F 1 "5V" H 1000 5049 40  0000 C CNN
+F 2 "~" H 1000 4900 60  0000 C CNN
+F 3 "~" H 1000 4900 60  0000 C CNN
+	1    1000 4900
+	1    0    0    -1
+$EndComp
+$Comp
+L 12V #PWR039
+U 1 1 571AE3BA
+P 750 4900
+F 0 "#PWR039" H 750 5000 40  0001 C CNN
+F 1 "12V" H 750 5049 40  0000 C CNN
+F 2 "~" H 750 4900 60  0000 C CNN
+F 3 "~" H 750 4900 60  0000 C CNN
+	1    750  4900
+	1    0    0    -1
+$EndComp
+$Comp
+L GND #PWR040
+U 1 1 571AE3C0
+P 1250 5200
+F 0 "#PWR040" H 1250 5200 30  0001 C CNN
+F 1 "GND" H 1250 5130 30  0001 C CNN
+F 2 "~" H 1250 5200 60  0000 C CNN
+F 3 "~" H 1250 5200 60  0000 C CNN
+	1    1250 5200
+	1    0    0    -1
+$EndComp
+Wire Wire Line
+	750  4950 750  4900
+Wire Wire Line
+	1000 4950 1000 4900
+Wire Wire Line
+	1250 5150 1250 5200
 $EndSCHEMATC

Commit message: work in progress
Parts:
- IC3: value MC9S12VRP64 -> MC9S12XXXXX; symbol MC9S12VRP64 -> MC9S12XXXXX
Changed lines of the file:
@@
 UART_TXD
 $Comp
-L MC9S12VRP64 IC3
+L MC9S12XXXXX IC3
 U 1 1 57040BB9
 P 6150 2400
 F 0 "IC3" H 6150 2500 60  0000 C CNN
-F 1 "MC9S12VRP64" H 6150 2300 60  0000 C CNN
+F 1 "MC9S12XXXXX" H 6150 2300 60  0000 C CNN
 F 2 "~" H 6700 2300 60  0000 C CNN
 F 3 "~" H 6700 2300 60  0000 C CNN
