File: Hardware/RevA/KiCad/MagniCube-RevA-UART.sch (KiCad schematic (older format))
At the start: 11 parts, among them CON2 USB-MINI-B, IC2 FT232RL

Commit message: schematic in progress
Parts:
- added C9: 100nF, ~, symbol C
- added D_VUSB1: SCHOTTKY, symbol SCHOTTKY
- added R4: 10k, ~, symbol R
- added R5: 4k7, ~, symbol R
- renumbered CON2 to CON3, LED3 to D_RXTX1
Connections:
- net labels added: VIO, VSUP
- net labels removed: 5V, VUSB
- wire segments 25 -> 32
- no-connect marks 18 -> 17
Other:
- moved on the sheet: C6, C7, C8
Changed lines of the file:
@@
 EESchema Schematic File Version 2
 LIBS:MagniCube
+LIBS:w_connectors
+LIBS:w_device
 LIBS:MagniCube-RevA-cache
 EELAYER 27 0
@@
 Sheet 2 4
 Title "UART"
-Date "5 apr 2016"
+Date "14 apr 2016"
 Rev "RevA"
 Comp "Dirk Heisswolf"
@@
 $EndComp
 $Comp
-L USB-MINI-B CON2
+L USB-MINI-B CON3
 U 1 1 544AC290
 P 2050 2300
-F 0 "CON2" H 2050 2750 60  0000 C CNN
+F 0 "CON3" H 2050 2750 60  0000 C CNN
 F 1 "USB-MINI-B" H 2000 1800 60  0000 C CNN
 F 2 "" H 2050 2300 60  0000 C CNN
@@
 NoConn ~ 4000 2800
 $Comp
-L GND #PWR018
+L GND #PWR_GND01
 U 1 1 54502C29
 P 4650 3900
-F 0 "#PWR018" H 4650 3900 30  0001 C CNN
+F 0 "#PWR_GND01" H 4650 3900 30  0001 C CNN
 F 1 "GND" H 4650 3830 30  0001 C CNN
 F 2 "" H 4650 3900 60  0000 C CNN
@@
 NoConn ~ 2600 2450
 $Comp
-L GND #PWR019
+L GND #PWR02
 U 1 1 54502C47
 P 2600 2700
-F 0 "#PWR019" H 2600 2700 30  0001 C CNN
+F 0 "#PWR02" H 2600 2700 30  0001 C CNN
 F 1 "GND" H 2600 2630 30  0001 C CNN
 F 2 "" H 2600 2700 60  0000 C CNN
@@
 $EndComp
 $Comp
-L GND #PWR020
+L GND #PWR_GND03
 U 1 1 54502C84
 P 3850 3550
-F 0 "#PWR020" H 3850 3550 30  0001 C CNN
+F 0 "#PWR_GND03" H 3850 3550 30  0001 C CNN
 F 1 "GND" H 3850 3480 30  0001 C CNN
 F 2 "" H 3850 3550 60  0000 C CNN
@@
 $EndComp
 $Comp
-L LED LED3
+L LED D_RXTX1
 U 1 1 54504211
 P 6750 2900
-F 0 "LED3" H 6750 3000 50  0000 C CNN
+F 0 "D_RXTX1" H 6750 3000 50  0000 C CNN
 F 1 "YELLOW" H 6700 2800 50  0000 C CNN
 F 2 "~" H 6750 2900 60  0000 C CNN
@@
 L C C6
 U 1 1 545042A7
-P 2400 1350
-F 0 "C6" H 2400 1450 40  0000 L CNN
-F 1 "10nF" H 2350 1250 40  0000 R CNN
-F 2 "~" H 2438 1200 30  0000 C CNN
-F 3 "~" H 2400 1350 60  0000 C CNN
-	1    2400 1350
+P 2600 1650
+F 0 "C6" H 2600 1750 40  0000 L CNN
+F 1 "10nF" H 2550 1550 40  0000 R CNN
+F 2 "~" H 2638 1500 30  0000 C CNN
+F 3 "~" H 2600 1650 60  0000 C CNN
+	1    2600 1650
 	1    0    0    -1
 $EndComp
@@
 L C C7
 U 1 1 545042B6
-P 3500 1350
-F 0 "C7" H 3500 1450 40  0000 L CNN
-F 1 "4.7uF" H 3506 1265 40  0000 L CNN
-F 2 "~" H 3538 1200 30  0000 C CNN
-F 3 "~" H 3500 1350 60  0000 C CNN
-	1    3500 1350
+P 1750 3550
+F 0 "C7" H 1750 3650 40  0000 L CNN
+F 1 "4.7uF" H 1756 3465 40  0000 L CNN
+F 2 "~" H 1788 3400 30  0000 C CNN
+F 3 "~" H 1750 3550 60  0000 C CNN
+	1    1750 3550
 	1    0    0    -1
 $EndComp
@@
 L C C8
 U 1 1 545042C5
-P 3700 1350
-F 0 "C8" H 3700 1450 40  0000 L CNN
-F 1 "100nF" H 3706 1265 40  0000 L CNN
-F 2 "~" H 3738 1200 30  0000 C CNN
-F 3 "~" H 3700 1350 60  0000 C CNN
-	1    3700 1350
-	1    0    0    -1
-$EndComp
-$Comp
-L GND #PWR022
+P 2050 3550
+F 0 "C8" H 2050 3650 40  0000 L CNN
+F 1 "100nF" H 2056 3465 40  0000 L CNN
+F 2 "~" H 2088 3400 30  0000 C CNN
+F 3 "~" H 2050 3550 60  0000 C CNN
+	1    2050 3550
+	1    0    0    -1
+$EndComp
+$Comp
+L GND #PWR_GND04
 U 1 1 545043BA
-P 2400 1600
-F 0 "#PWR022" H 2400 1600 30  0001 C CNN
-F 1 "GND" H 2400 1530 30  0001 C CNN
-F 2 "" H 2400 1600 60  0000 C CNN
-F 3 "" H 2400 1600 60  0000 C CNN
-	1    2400 1600
-	1    0    0    -1
-$EndComp
-$Comp
-L GND #PWR023
+P 2450 1550
+F 0 "#PWR_GND04" H 2450 1550 30  0001 C CNN
+F 1 "GND" H 2450 1480 30  0001 C CNN
+F 2 "" H 2450 1550 60  0000 C CNN
+F 3 "" H 2450 1550 60  0000 C CNN
+	1    2450 1550
+	1    0    0    -1
+$EndComp
+$Comp
+L GND #PWR_GND05
 U 1 1 545043C9
-P 3600 1600
-F 0 "#PWR023" H 3600 1600 30  0001 C CNN
-F 1 "GND" H 3600 1530 30  0001 C CNN
-F 2 "" H 3600 1600 60  0000 C CNN
-F 3 "" H 3600 1600 60  0000 C CNN
-	1    3600 1600
-	1    0    0    -1
-$EndComp
-$Comp
-L VUSB #PWR024
-U 1 1 54504942
-P 3400 1150
-F 0 "#PWR024" H 3400 1100 20  0001 C CNN
-F 1 "VUSB" H 3400 1250 30  0000 C CNN
-F 2 "" H 3400 1150 60  0000 C CNN
-F 3 "" H 3400 1150 60  0000 C CNN
-	1    3400 1150
-	1    0    0    -1
-$EndComp
-Wire Wire Line
-	4650 3800 5250 3800
-Connection ~ 4800 3800
-Connection ~ 5100 3800
-Connection ~ 4950 3800
-Wire Wire Line
-	4650 3800 4650 3900
-Wire Wire Line
-	2600 2600 2600 2700
-Wire Wire Line
-	3850 3500 3850 3550
-Wire Wire Line
-	4000 1950 3400 1950
-Wire Wire Line
-	4000 2300 2600 2300
-Wire Wire Line
-	4000 2200 2600 2200
-Wire Wire Line
-	2600 2200 2600 2150
-Wire Wire Line
-	2700 1950 2600 1950
-Wire Wire Line
-	2600 1150 2600 2000
-Wire Wire Line
-	2600 1150 2400 1150
-Connection ~ 2600 1950
-Wire Wire Line
-	3400 1950 3400 1150
-Wire Wire Line
-	3400 1150 3700 1150
-Connection ~ 3500 1150
-Wire Wire Line
-	3500 1550 3700 1550
-Wire Wire Line
-	2400 1550 2400 1600
-Wire Wire Line
-	3600 1550 3600 1600
-Connection ~ 3600 1550
+P 3500 3550
+F 0 "#PWR_GND05" H 3500 3550 30  0001 C CNN
+F 1 "GND" H 3500 3480 30  0001 C CNN
+F 2 "" H 3500 3550 60  0000 C CNN
+F 3 "" H 3500 3550 60  0000 C CNN
+	1    3500 3550
+	1    0    0    -1
+$EndComp
 Text Label 2650 2300 0    60   ~ 0
 USBD+
@@
 NoConn ~ 1500 2450
 NoConn ~ 1500 2600
-NoConn ~ 4000 2600
-Wire Wire Line
-	4000 3100 3850 3100
-Connection ~ 4000 1850
-Wire Wire Line
-	5850 2900 5950 2900
-Wire Wire Line
-	6450 2900 6550 2900
-Wire Wire Line
-	4000 1700 4000 1950
-$Comp
-L 5V #PWR?
+$Comp
+L 5V #PWR_IO2
 U 1 1 5703751E
-P 4000 1700
-F 0 "#PWR?" H 4000 1800 40  0001 C CNN
-F 1 "5V" H 4000 1849 40  0000 C CNN
-F 2 "~" H 4000 1700 60  0000 C CNN
-F 3 "~" H 4000 1700 60  0000 C CNN
-	1    4000 1700
-	1    0    0    -1
-$EndComp
-$Comp
-L 5V #PWR?
+P 4000 1800
+F 0 "#PWR_IO2" H 4000 1900 40  0001 C CNN
+F 1 "VIO" H 4000 1949 40  0000 C CNN
+F 2 "~" H 4000 1800 60  0000 C CNN
+F 3 "~" H 4000 1800 60  0000 C CNN
+	1    4000 1800
+	1    0    0    -1
+$EndComp
+$Comp
+L 5V #PWR_IO3
 U 1 1 5703752D
 P 6950 2750
-F 0 "#PWR?" H 6950 2850 40  0001 C CNN
-F 1 "5V" H 6950 2899 40  0000 C CNN
+F 0 "#PWR_IO3" H 6950 2850 40  0001 C CNN
+F 1 "VIO" H 6950 2899 40  0000 C CNN
 F 2 "~" H 6950 2750 60  0000 C CNN
 F 3 "~" H 6950 2750 60  0000 C CNN
@@
 	1    0    0    -1
 $EndComp
-Wire Wire Line
-	6950 2750 6950 2900
 Text GLabel 6550 1900 2    39   Output ~ 0
 UART_RXD
@@
 	0    1    -1   0
 $EndComp
+$Comp
+L C C9
+U 1 1 570D12A2
+P 2350 3550
+F 0 "C9" H 2350 3650 40  0000 L CNN
+F 1 "100nF" H 2356 3465 40  0000 L CNN
+F 2 "~" H 2388 3400 30  0000 C CNN
+F 3 "~" H 2350 3550 60  0000 C CNN
+	1    2350 3550
+	1    0    0    -1
+$EndComp
+$Comp
+L 5V #PWR_IO1
+U 1 1 570D1336
+P 2050 3250
+F 0 "#PWR_IO1" H 2050 3350 40  0001 C CNN
+F 1 "VIO" H 2050 3399 40  0000 C CNN
+F 2 "~" H 2050 3250 60  0000 C CNN
+F 3 "~" H 2050 3250 60  0000 C CNN
+	1    2050 3250
+	1    0    0    -1
+$EndComp
+$Comp
+L R R4
+U 1 1 570D133E
+P 3500 3250
+F 0 "R4" V 3580 3250 40  0000 C CNN
+F 1 "10k" V 3507 3251 40  0000 C CNN
+F 2 "~" V 3430 3250 30  0000 C CNN
+F 3 "~" H 3500 3250 30  0000 C CNN
+	1    3500 3250
+	1    0    0    -1
+$EndComp
+$Comp
+L R R5
+U 1 1 570D134D
+P 3500 2650
+F 0 "R5" V 3580 2650 40  0000 C CNN
+F 1 "4k7" V 3507 2651 40  0000 C CNN
+F 2 "~" V 3430 2650 30  0000 C CNN
+F 3 "~" H 3500 2650 30  0000 C CNN
+	1    3500 2650
+	1    0    0    -1
+$EndComp
+$Comp
+L SCHOTTKY D_VUSB1
+U 1 1 570D83A1
+P 3500 1800
+F 0 "D_VUSB1" H 3500 1900 40  0000 C CNN
+F 1 "SCHOTTKY" H 3500 1700 40  0000 C CNN
+F 2 "" H 3500 1800 60  0000 C CNN
+F 3 "" H 3500 1800 60  0000 C CNN
+	1    3500 1800
+	0    -1   -1   0
+$EndComp
+$Comp
+L 12V #PWR_SUPPLY1
+U 1 1 570D83B0
+P 3500 1600
+F 0 "#PWR_SUPPLY1" H 3500 1700 40  0001 C CNN
+F 1 "VSUP" H 3500 1749 40  0000 C CNN
+F 2 "~" H 3500 1600 60  0000 C CNN
+F 3 "~" H 3500 1600 60  0000 C CNN
+	1    3500 1600
+	1    0    0    -1
+$EndComp
+$Comp
+L GND #PWR_GND06
+U 1 1 570D8434
+P 2050 3850
+F 0 "#PWR_GND06" H 2050 3850 30  0001 C CNN
+F 1 "GND" H 2050 3780 30  0001 C CNN
+F 2 "" H 2050 3850 60  0000 C CNN
+F 3 "" H 2050 3850 60  0000 C CNN
+	1    2050 3850
+	1    0    0    -1
+$EndComp
+Wire Wire Line
+	4650 3800 5250 3800
+Connection ~ 4800 3800
+Connection ~ 5100 3800
+Connection ~ 4950 3800
+Wire Wire Line
+	4650 3800 4650 3900
+Wire Wire Line
+	2600 2600 2600 2700
+Wire Wire Line
+	3850 3500 3850 3550
+Wire Wire Line
+	4000 2300 2600 2300
+Wire Wire Line
+	4000 2200 2600 2200
+Wire Wire Line
+	2600 2200 2600 2150
+Wire Wire Line
+	2700 1950 2600 1950
+Connection ~ 2600 1950
+Wire Wire Line
+	4000 3100 3850 3100
+Connection ~ 4000 1850
+Wire Wire Line
+	5850 2900 5950 2900
+Wire Wire Line
+	6450 2900 6550 2900
+Wire Wire Line
+	6950 2750 6950 2900
 Wire Wire Line
 	5850 1900 5950 1900
@@
 Wire Wire Line
 	6450 2000 6550 2000
+Wire Wire Line
+	4000 1800 4000 1950
+Wire Wire Line
+	3400 1950 3500 1950
+Wire Wire Line
+	3500 1850 3500 2400
+Wire Wire Line
+	3500 2900 3500 3000
+Wire Wire Line
+	3500 3500 3500 3550
+Wire Wire Line
+	3500 2900 3700 2900
+Wire Wire Line
+	3700 2900 3700 2600
+Wire Wire Line
+	3700 2600 4000 2600
+Connection ~ 3500 2900
+Wire Wire Line
+	2600 1850 2600 2000
+Wire Wire Line
+	2600 1450 2450 1450
+Wire Wire Line
+	2450 1450 2450 1550
+Connection ~ 3500 1950
+Wire Wire Line
+	3500 1700 3500 1600
+Wire Wire Line
+	1750 3750 2350 3750
+Connection ~ 2050 3750
+Wire Wire Line
+	1750 3350 2350 3350
+Connection ~ 2050 3350
+Wire Wire Line
+	2050 3350 2050 3250
+Wire Wire Line
+	2050 3750 2050 3850
 $EndSCHEMATC

Commit message: PCB in progress
Parts:
- renumbered C7 to C1, C8 to C2, C9 to C3, C5 to C4, C6 to C5, CON3 to CON1, IC2 to IC1
Changed lines of the file:
@@
 Sheet 2 4
 Title "UART"
-Date "14 apr 2016"
+Date "18 apr 2016"
 Rev "RevA"
 Comp "Dirk Heisswolf"
@@
 $EndDescr
 $Comp
-L FT232RL IC2
+L FT232RL IC1
 U 1 1 544AC281
 P 4950 2600
-F 0 "IC2" H 4950 3500 60  0000 C CNN
+F 0 "IC1" H 4950 3500 60  0000 C CNN
 F 1 "FT232RL" H 5350 1600 60  0000 L CNN
 F 2 "" H 4950 2600 60  0000 C CNN
@@
 $EndComp
 $Comp
-L USB-MINI-B CON3
+L USB-MINI-B CON1
 U 1 1 544AC290
 P 2050 2300
-F 0 "CON3" H 2050 2750 60  0000 C CNN
+F 0 "CON1" H 2050 2750 60  0000 C CNN
 F 1 "USB-MINI-B" H 2000 1800 60  0000 C CNN
 F 2 "" H 2050 2300 60  0000 C CNN
@@
 NoConn ~ 5850 3100
 $Comp
-L C C5
+L C C4
 U 1 1 54502C6B
 P 3850 3300
-F 0 "C5" H 3850 3400 40  0000 L CNN
+F 0 "C4" H 3850 3400 40  0000 L CNN
 F 1 "100nF" H 3856 3215 40  0000 L CNN
 F 2 "~" H 3888 3150 30  0000 C CNN
@@
 $EndComp
 $Comp
-L C C6
+L C C5
 U 1 1 545042A7
 P 2600 1650
-F 0 "C6" H 2600 1750 40  0000 L CNN
+F 0 "C5" H 2600 1750 40  0000 L CNN
 F 1 "10nF" H 2550 1550 40  0000 R CNN
 F 2 "~" H 2638 1500 30  0000 C CNN
@@
 $EndComp
 $Comp
-L C C7
+L C C1
 U 1 1 545042B6
 P 1750 3550
-F 0 "C7" H 1750 3650 40  0000 L CNN
+F 0 "C1" H 1750 3650 40  0000 L CNN
 F 1 "4.7uF" H 1756 3465 40  0000 L CNN
 F 2 "~" H 1788 3400 30  0000 C CNN
@@
 $EndComp
 $Comp
-L C C8
+L C C2
 U 1 1 545042C5
 P 2050 3550
-F 0 "C8" H 2050 3650 40  0000 L CNN
+F 0 "C2" H 2050 3650 40  0000 L CNN
 F 1 "100nF" H 2056 3465 40  0000 L CNN
 F 2 "~" H 2088 3400 30  0000 C CNN
@@
 $EndComp
 $Comp
-L C C9
+L C C3
 U 1 1 570D12A2
 P 2350 3550
-F 0 "C9" H 2350 3650 40  0000 L CNN
+F 0 "C3" H 2350 3650 40  0000 L CNN
 F 1 "100nF" H 2356 3465 40  0000 L CNN
 F 2 "~" H 2388 3400 30  0000 C CNN

Commit message: work in progress
Parts:
- removed R2, R3: 100, ~, symbol R
- renumbered R4 to R2, R5 to R3
Connections:
- net UART_RXD: now also IC1.1 (TXD)
- net UART_TXD: now also IC1.5 (RXD)
Changed lines of the file:
@@
 Sheet 2 4
 Title "UART"
-Date "18 apr 2016"
+Date "19 apr 2016"
 Rev "RevA"
 Comp "Dirk Heisswolf"
@@
 NoConn ~ 4000 2800
 $Comp
-L GND #PWR_GND01
+L GND #PWR?
 U 1 1 54502C29
 P 4650 3900
-F 0 "#PWR_GND01" H 4650 3900 30  0001 C CNN
+F 0 "#PWR?" H 4650 3900 30  0001 C CNN
 F 1 "GND" H 4650 3830 30  0001 C CNN
 F 2 "" H 4650 3900 60  0000 C CNN
@@
 NoConn ~ 2600 2450
 $Comp
-L GND #PWR02
+L GND #PWR?
 U 1 1 54502C47
 P 2600 2700
-F 0 "#PWR02" H 2600 2700 30  0001 C CNN
+F 0 "#PWR?" H 2600 2700 30  0001 C CNN
 F 1 "GND" H 2600 2630 30  0001 C CNN
 F 2 "" H 2600 2700 60  0000 C CNN
@@
 $EndComp
 $Comp
-L GND #PWR_GND03
+L GND #PWR?
 U 1 1 54502C84
 P 3850 3550
-F 0 "#PWR_GND03" H 3850 3550 30  0001 C CNN
+F 0 "#PWR?" H 3850 3550 30  0001 C CNN
 F 1 "GND" H 3850 3480 30  0001 C CNN
 F 2 "" H 3850 3550 60  0000 C CNN
@@
 $EndComp
 $Comp
-L GND #PWR_GND04
+L GND #PWR?
 U 1 1 545043BA
 P 2450 1550
-F 0 "#PWR_GND04" H 2450 1550 30  0001 C CNN
+F 0 "#PWR?" H 2450 1550 30  0001 C CNN
 F 1 "GND" H 2450 1480 30  0001 C CNN
 F 2 "" H 2450 1550 60  0000 C CNN
@@
 $EndComp
 $Comp
-L GND #PWR_GND05
+L GND #PWR?
 U 1 1 545043C9
 P 3500 3550
-F 0 "#PWR_GND05" H 3500 3550 30  0001 C CNN
+F 0 "#PWR?" H 3500 3550 30  0001 C CNN
 F 1 "GND" H 3500 3480 30  0001 C CNN
 F 2 "" H 3500 3550 60  0000 C CNN
@@
 	1    0    0    -1
 $EndComp
-Text GLabel 6550 1900 2    39   Output ~ 0
+Text GLabel 6100 1900 2    39   Output ~ 0
 UART_RXD
-Text GLabel 6550 2000 2    39   Input ~ 0
+Text GLabel 6100 2000 2    39   Input ~ 0
 UART_TXD
-$Comp
-L R R3
-U 1 1 57040E44
-P 6200 2000
-F 0 "R3" V 6280 2000 40  0000 C CNN
-F 1 "100" V 6207 2001 40  0000 C CNN
-F 2 "~" V 6130 2000 30  0000 C CNN
-F 3 "~" H 6200 2000 30  0000 C CNN
-	1    6200 2000
-	0    1    1    0
-$EndComp
-$Comp
-L R R2
-U 1 1 57040E4A
-P 6200 1900
-F 0 "R2" V 6280 1900 40  0000 C CNN
-F 1 "100" V 6207 1901 40  0000 C CNN
-F 2 "~" V 6130 1900 30  0000 C CNN
-F 3 "~" H 6200 1900 30  0000 C CNN
-	1    6200 1900
-	0    1    -1   0
-$EndComp
 $Comp
 L C C3
@@
 $EndComp
 $Comp
-L R R4
+L R R2
 U 1 1 570D133E
 P 3500 3250
-F 0 "R4" V 3580 3250 40  0000 C CNN
+F 0 "R2" V 3580 3250 40  0000 C CNN
 F 1 "10k" V 3507 3251 40  0000 C CNN
 F 2 "~" V 3430 3250 30  0000 C CNN
@@
 $EndComp
 $Comp
-L R R5
+L R R3
 U 1 1 570D134D
 P 3500 2650
-F 0 "R5" V 3580 2650 40  0000 C CNN
+F 0 "R3" V 3580 2650 40  0000 C CNN
 F 1 "4k7" V 3507 2651 40  0000 C CNN
 F 2 "~" V 3430 2650 30  0000 C CNN
@@
 $EndComp
 $Comp
-L GND #PWR_GND06
+L GND #PWR?
 U 1 1 570D8434
 P 2050 3850
-F 0 "#PWR_GND06" H 2050 3850 30  0001 C CNN
+F 0 "#PWR?" H 2050 3850 30  0001 C CNN
 F 1 "GND" H 2050 3780 30  0001 C CNN
 F 2 "" H 2050 3850 60  0000 C CNN
@@
 	6950 2750 6950 2900
 Wire Wire Line
-	5850 1900 5950 1900
-Wire Wire Line
-	5850 2000 5950 2000
-Wire Wire Line
-	6450 1900 6550 1900
-Wire Wire Line
-	6450 2000 6550 2000
+	5850 1900 6100 1900
+Wire Wire Line
+	5850 2000 6100 2000
 Wire Wire Line
 	4000 1800 4000 1950

Commit message: work in progress
Changed lines of the file:
@@
 Sheet 2 4
 Title "UART"
-Date "19 apr 2016"
+Date "20 apr 2016"
 Rev "RevA"
 Comp "Dirk Heisswolf"
@@
 	1    0    0    -1
 $EndComp
-Text Label 2650 2300 0    60   ~ 0
+Text Label 2650 2300 0    39   ~ 0
 USBD+
-Text Label 2650 2200 0    60   ~ 0
+Text Label 2650 2200 0    39   ~ 0
 USBD-
 NoConn ~ 5850 2200
@@
 NoConn ~ 1500 2450
 NoConn ~ 1500 2600
-$Comp
-L 5V #PWR_IO2
-U 1 1 5703751E
-P 4000 1800
-F 0 "#PWR_IO2" H 4000 1900 40  0001 C CNN
-F 1 "VIO" H 4000 1949 40  0000 C CNN
-F 2 "~" H 4000 1800 60  0000 C CNN
-F 3 "~" H 4000 1800 60  0000 C CNN
-	1    4000 1800
-	1    0    0    -1
-$EndComp
-$Comp
-L 5V #PWR_IO3
-U 1 1 5703752D
-P 6950 2750
-F 0 "#PWR_IO3" H 6950 2850 40  0001 C CNN
-F 1 "VIO" H 6950 2899 40  0000 C CNN
-F 2 "~" H 6950 2750 60  0000 C CNN
-F 3 "~" H 6950 2750 60  0000 C CNN
-	1    6950 2750
-	1    0    0    -1
-$EndComp
 Text GLabel 6100 1900 2    39   Output ~ 0
 UART_RXD
@@
 F 3 "~" H 2350 3550 60  0000 C CNN
 	1    2350 3550
-	1    0    0    -1
-$EndComp
-$Comp
-L 5V #PWR_IO1
-U 1 1 570D1336
-P 2050 3250
-F 0 "#PWR_IO1" H 2050 3350 40  0001 C CNN
-F 1 "VIO" H 2050 3399 40  0000 C CNN
-F 2 "~" H 2050 3250 60  0000 C CNN
-F 3 "~" H 2050 3250 60  0000 C CNN
-	1    2050 3250
 	1    0    0    -1
 $EndComp
@@
 $EndComp
 $Comp
-L 12V #PWR_SUPPLY1
-U 1 1 570D83B0
-P 3500 1600
-F 0 "#PWR_SUPPLY1" H 3500 1700 40  0001 C CNN
-F 1 "VSUP" H 3500 1749 40  0000 C CNN
-F 2 "~" H 3500 1600 60  0000 C CNN
-F 3 "~" H 3500 1600 60  0000 C CNN
-	1    3500 1600
-	1    0    0    -1
-$EndComp
-$Comp
 L GND #PWR?
 U 1 1 570D8434
@@
 	6450 2900 6550 2900
 Wire Wire Line
-	6950 2750 6950 2900
-Wire Wire Line
 	5850 1900 6100 1900
 Wire Wire Line
 	5850 2000 6100 2000
-Wire Wire Line
-	4000 1800 4000 1950
 Wire Wire Line
 	3400 1950 3500 1950
@@
 Connection ~ 3500 1950
 Wire Wire Line
-	3500 1700 3500 1600
-Wire Wire Line
 	1750 3750 2350 3750
 Connection ~ 2050 3750
@@
 Connection ~ 2050 3350
 Wire Wire Line
-	2050 3350 2050 3250
-Wire Wire Line
 	2050 3750 2050 3850
+Text Label 2350 3750 2    39   ~ 0
+GND
+Text Label 2600 2600 0    39   ~ 0
+GND
+Text Label 3500 3550 1    39   ~ 0
+GND
+Text Label 3850 3550 1    39   ~ 0
+GND
+Text Label 5250 3800 2    39   ~ 0
+GND
+Text Label 2600 1450 2    39   ~ 0
+GND
+$Comp
+L 5V #PWR?
+U 1 1 57181667
+P 2050 3300
+F 0 "#PWR?" H 2050 3400 40  0001 C CNN
+F 1 "5V" H 2050 3449 40  0000 C CNN
+F 2 "~" H 2050 3300 60  0000 C CNN
+F 3 "~" H 2050 3300 60  0000 C CNN
+	1    2050 3300
+	1    0    0    -1
+$EndComp
+Wire Wire Line
+	2050 3300 2050 3350
+Text Label 4000 1850 3    39   ~ 0
+5V
+Text Label 2350 3350 2    39   ~ 0
+5V
+$Comp
+L 5V #PWR?
+U 1 1 57181697
+P 4000 1800
+F 0 "#PWR?" H 4000 1900 40  0001 C CNN
+F 1 "5V" H 4000 1949 40  0000 C CNN
+F 2 "~" H 4000 1800 60  0000 C CNN
+F 3 "~" H 4000 1800 60  0000 C CNN
+	1    4000 1800
+	1    0    0    -1
+$EndComp
+Wire Wire Line
+	4000 1800 4000 1950
+$Comp
+L 12V #PWR?
+U 1 1 571816F0
+P 3500 1600
+F 0 "#PWR?" H 3500 1700 40  0001 C CNN
+F 1 "12V" H 3500 1749 40  0000 C CNN
+F 2 "~" H 3500 1600 60  0000 C CNN
+F 3 "~" H 3500 1600 60  0000 C CNN
+	1    3500 1600
+	1    0    0    -1
+$EndComp
+Text Label 3500 1600 3    39   ~ 0
+12V
+Wire Wire Line
+	3500 1600 3500 1700
+$Comp
+L 5V #PWR?
+U 1 1 57181745
+P 6950 2800
+F 0 "#PWR?" H 6950 2900 40  0001 C CNN
+F 1 "5V" H 6950 2949 40  0000 C CNN
+F 2 "~" H 6950 2800 60  0000 C CNN
+F 3 "~" H 6950 2800 60  0000 C CNN
+	1    6950 2800
+	1    0    0    -1
+$EndComp
+Wire Wire Line
+	6950 2800 6950 2900
+Text Label 6950 2900 1    39   ~ 0
+5V
 $EndSCHEMATC

Commit message: work in progress
Parts:
- renumbered D_VUSB1 to D2
Connections:
- no-connect marks 17 -> 13

Commit message: work in progress
Connections:
- no-connect marks 13 -> 17
Changed lines of the file:
@@
 Sheet 2 4
 Title "UART"
-Date "22 apr 2016"
+Date "23 apr 2016"
 Rev "RevA"
 Comp "Dirk Heisswolf"
@@
 UART_TXD
 $Comp
-L C C3
-U 1 1 570D12A2
-P 2350 3550
-F 0 "C3" H 2350 3650 40  0000 L CNN
-F 1 "100nF" H 2356 3465 40  0000 L CNN
-F 2 "~" H 2388 3400 30  0000 C CNN
-F 3 "~" H 2350 3550 60  0000 C CNN
-	1    2350 3550
-	1    0    0    -1
-$EndComp
-$Comp
 L R R2
 U 1 1 570D133E
@@
 Wire Wire Line
 	2050 3750 2050 3850
-Text Label 2350 3750 2    39   ~ 0
-GND
-Text Label 2600 2600 0    39   ~ 0
-GND
-Text Label 3500 3550 1    39   ~ 0
-GND
-Text Label 3850 3550 1    39   ~ 0
-GND
-Text Label 5250 3800 2    39   ~ 0
-GND
-Text Label 2600 1450 2    39   ~ 0
-GND
-$Comp
-L 5V #PWR1
+$Comp
+L 5V #PWR07
 U 1 1 57181667
 P 2050 3300
-F 0 "#PWR1" H 2050 3400 40  0001 C CNN
+F 0 "#PWR07" H 2050 3400 40  0001 C CNN
 F 1 "5V" H 2050 3449 40  0000 C CNN
 F 2 "~" H 2050 3300 60  0000 C CNN
@@
 	1    0    0    -1
 $EndComp
-Wire Wire Line
-	2050 3300 2050 3350
-Text Label 4000 1850 3    39   ~ 0
-5V
-Text Label 2350 3350 2    39   ~ 0
-5V
-$Comp
-L 5V #PWR8
+$Comp
+L 5V #PWR08
 U 1 1 57181697
 P 4000 1800
-F 0 "#PWR8" H 4000 1900 40  0001 C CNN
+F 0 "#PWR08" H 4000 1900 40  0001 C CNN
 F 1 "5V" H 4000 1949 40  0000 C CNN
 F 2 "~" H 4000 1800 60  0000 C CNN
@@
 	4000 1800 4000 1950
 $Comp
-L 12V #PWR5
+L 12V #PWR09
 U 1 1 571816F0
-P 3500 1600
-F 0 "#PWR5" H 3500 1700 40  0001 C CNN
-F 1 "12V" H 3500 1749 40  0000 C CNN
-F 2 "~" H 3500 1600 60  0000 C CNN
-F 3 "~" H 3500 1600 60  0000 C CNN
-	1    3500 1600
-	1    0    0    -1
-$EndComp
-Text Label 3500 1600 3    39   ~ 0
-12V
-Wire Wire Line
-	3500 1600 3500 1700
-$Comp
-L 5V #PWR10
+P 3500 1650
+F 0 "#PWR09" H 3500 1750 40  0001 C CNN
+F 1 "12V" H 3500 1799 40  0000 C CNN
+F 2 "~" H 3500 1650 60  0000 C CNN
+F 3 "~" H 3500 1650 60  0000 C CNN
+	1    3500 1650
+	1    0    0    -1
+$EndComp
+Wire Wire Line
+	3500 1650 3500 1700
+$Comp
+L 5V #PWR010
 U 1 1 57181745
 P 6950 2800
-F 0 "#PWR10" H 6950 2900 40  0001 C CNN
+F 0 "#PWR010" H 6950 2900 40  0001 C CNN
 F 1 "5V" H 6950 2949 40  0000 C CNN
 F 2 "~" H 6950 2800 60  0000 C CNN
@@
 Wire Wire Line
 	6950 2800 6950 2900
-Text Label 6950 2900 1    39   ~ 0
-5V
 $Comp
 L USB-MINI-B CON1
@@
 	-1   0    0    -1
 $EndComp
+$Comp
+L C C3
+U 1 1 570D12A2
+P 2350 3550
+F 0 "C3" H 2350 3650 40  0000 L CNN
+F 1 "100nF" H 2356 3465 40  0000 L CNN
+F 2 "~" H 2388 3400 30  0000 C CNN
+F 3 "~" H 2350 3550 60  0000 C CNN
+	1    2350 3550
+	1    0    0    -1
+$EndComp
+Wire Wire Line
+	2050 3350 2050 3300
+NoConn ~ 1500 2000
+NoConn ~ 1500 2150
+NoConn ~ 1500 2450
+NoConn ~ 1500 2600
 $EndSCHEMATC

Commit message: work in progress
Parts:
- added SG1, SG2, SG3, SG4: SPARK_GAP, symbol SPARK_GAP
Connections:
- net at CON1.6 (SHELL1): now also SG1.~
- net at CON1.7 (SHELL2): now also SG2.~
- net at CON1.8 (SHELL3): now also SG3.~
- net at CON1.9 (SHELL4): now also SG4.~
- no-connect marks 17 -> 13
Changed lines of the file:
@@
 Wire Wire Line
 	2050 3350 2050 3300
-NoConn ~ 1500 2000
-NoConn ~ 1500 2150
-NoConn ~ 1500 2450
-NoConn ~ 1500 2600
+$Comp
+L SPARK_GAP SG1
+U 1 1 571C0840
+P 1450 2000
+F 0 "SG1" H 1400 2100 60  0001 C CNN
+F 1 "SPARK_GAP" H 1400 1900 60  0001 C CNN
+F 2 "" H 1450 2000 60  0000 C CNN
+F 3 "" H 1450 2000 60  0000 C CNN
+	1    1450 2000
+	1    0    0    -1
+$EndComp
+$Comp
+L SPARK_GAP SG2
+U 1 1 571C084D
+P 1450 2150
+F 0 "SG2" H 1400 2250 60  0001 C CNN
+F 1 "SPARK_GAP" H 1400 2050 60  0001 C CNN
+F 2 "" H 1450 2150 60  0000 C CNN
+F 3 "" H 1450 2150 60  0000 C CNN
+	1    1450 2150
+	1    0    0    -1
+$EndComp
+$Comp
+L SPARK_GAP SG3
+U 1 1 571C0853
+P 1450 2450
+F 0 "SG3" H 1400 2550 60  0001 C CNN
+F 1 "SPARK_GAP" H 1400 2350 60  0001 C CNN
+F 2 "" H 1450 2450 60  0000 C CNN
+F 3 "" H 1450 2450 60  0000 C CNN
+	1    1450 2450
+	1    0    0    -1
+$EndComp
+$Comp
+L SPARK_GAP SG4
+U 1 1 571C0859
+P 1450 2600
+F 0 "SG4" H 1400 2700 60  0001 C CNN
+F 1 "SPARK_GAP" H 1400 2500 60  0001 C CNN
+F 2 "" H 1450 2600 60  0000 C CNN
+F 3 "" H 1450 2600 60  0000 C CNN
+	1    1450 2600
+	1    0    0    -1
+$EndComp
+Wire Wire Line
+	1500 2000 1450 2000
+Wire Wire Line
+	1500 2150 1450 2150
+Wire Wire Line
+	1500 2450 1450 2450
+Wire Wire Line
+	1500 2600 1450 2600
 $EndSCHEMATC
